File: Decoder/Decoder.kicad_pcb (KiCad board)
At the start: 2 copper layers, 272.4 x 146.7 mm, 198 parts, among them J4A1 EdgeTop, J4B1 EdgeBottom, J981 USB_B, Q1 2N2369A, Q2 2N2369A, Q901 2N7002, Q902 2N7002, Q903 2N7002, Q904 2N7002, Q905 2N7002, SW981 BOOTSEL, SW982 RUN STOP, SW983 +/T, SW984 -/S, U901 74HCT245, U902 74HCT245, U941 74LS04, U942 74LS04, U943 74LS04, U944 74LS04, U981 RP2040_Stamp, U982 74LVC245, Y1 9.8400MHz

Commit message: Schematics for display & keyboard, adding LEDs to processor PCB
Parts:
- added H907: MountingHole, MountingHole:MountingHole_3.2mm_M3, F.Cu at (156.2, 18.4)
- added H908: MountingHole, MountingHole:MountingHole_3.2mm_M3, F.Cu at (156.2, 156.2)
- added J902: ~WORD_SELECT, Connector_PinHeader_2.54mm:PinHeader_1x01_P2.54mm_Horizontal, F.Cu at (236.9, 64.1)
- added Q906: 2N7002, Package_TO_SOT_SMD:SOT-23, B.Cu at (239.4, 56.5)
- D902: value S0 -> C3
- D903: value S3 -> C0
- D904: value S1 -> C2
- D905: value S2 -> C1
- D941: value PORT8 -> PORT0
- D942: value PORT9 -> PORT1
- D943: value PORT10 -> PORT2
- D944: value PORT11 -> PORT3
- R1, R10, R11, R12, R13, R14, R15, R16, R17, R18, R19, R2, R20, R21, R22, R23, R24, R25, R26, R27, R28, R3, R4, R5, R6, R7, R8, R9: footprint Resistor_THT:R_Axial_DIN0207_L6.3mm_D2.5mm_P7.62mm_Horizontal -> Resistor_THT:R_Axial_DIN0207_L6.3mm_D2.5mm_P10.16mm_Horizontal
- Z14, Z21: footprint Package_DIP:DIP-24_W10.16mm_Socket -> Package_DIP:DIP-24_W15.24mm_Socket
- moved SW981 34.2 mm to (265.9, 65.1), turned to 0 degrees
- moved Q905 16.0 mm to (126.5, 59.8)
- moved R5 6.98 mm to (243.2, 66.0), turned to 270 degrees
- moved D921 6.35 mm to (65.8, 19.1)
- moved R921 6.35 mm to (69.1, 21.3)
- moved D916 5.72 mm to (98.2, 19.1)
- moved D918 5.72 mm to (83.0, 19.1)
- moved D920 5.72 mm to (90.6, 19.1)
- moved R919 5.72 mm to (79.1, 23.4)
- moved D919 5.71 mm to (75.4, 19.1)
- moved D917 5.08 mm to (107.7, 19.1)
- moved D903 4.45 mm to (208.7, 19.1)
- moved D908 4.45 mm to (189.0, 19.1)
- moved R907 4.45 mm to (176.9, 23.9)
- moved D913 4.45 mm to (116.6, 19.1)
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Connections:
- net S0 renamed C0
- net S1 renamed C1
- net S2 renamed C2
- net ~I1 renamed I1
- net ~I2 renamed I2
- net ~I3 renamed I3
- net ~I4 renamed I4
- net ~PORT10 renamed ~PORT2
- net ~PORT11 renamed ~PORT3
- net ~PORT8 renamed ~PORT0
- net ~PORT9 renamed ~PORT1
- Q905 pad 1: DIV64_CLK -> C3
- R902 pad 2: /Scheduler/StampClock/S0 -> /Scheduler/StampClock/C3
- R903 pad 2: /Scheduler/StampClock/S3 -> /Scheduler/StampClock/C0
- R904 pad 2: /Scheduler/StampClock/S1 -> /Scheduler/StampClock/C2
- R905 pad 2: /Scheduler/StampClock/S2 -> /Scheduler/StampClock/C1
- U901 pad 15: /Scheduler/StampClock/S3 -> /Scheduler/StampClock/C3
- U901 pad 16: /Scheduler/StampClock/S2 -> /Scheduler/StampClock/C2
- U901 pad 17: /Scheduler/StampClock/S1 -> /Scheduler/StampClock/C1
- U901 pad 18: /Scheduler/StampClock/S0 -> /Scheduler/StampClock/C0
- U901 pad 5: S3 -> C3
- U981 pad 10: Net-(U981-Pad10) -> WORD_SELECT
- U982 pad 2: /Scheduler/StampClock/S3 -> /Scheduler/StampClock/C3
- U982 pad 3: /Scheduler/StampClock/S2 -> /Scheduler/StampClock/C2
- U982 pad 4: /Scheduler/StampClock/S1 -> /Scheduler/StampClock/C1
- U982 pad 5: /Scheduler/StampClock/S0 -> /Scheduler/StampClock/C0
- Z13 pad 3: S3 -> C3
- Z15 pad 13: S3 -> C3
- Z17 pad 12: S3 -> C3
- Z2 pad 11: S3 -> C3
- Z3 pad 6: S3 -> C3
- Z3 pad 8: S3 -> C3
- Z7 pad 4: S3 -> C3
- Z7 pad 9: S3 -> C3
Routing:
- net S3: track 262.8 -> 0.00 mm, vias 2 -> 0
- net C3: track 0.00 -> 261.4 mm, vias 0 -> 2
- net /Scheduler/StampClock/C3: track 0.00 -> 44.9 mm
- net /Scheduler/StampClock/C2: track 0.00 -> 42.8 mm
- net /Scheduler/StampClock/C1: track 0.00 -> 42.0 mm
- net /Scheduler/StampClock/S3: track 41.2 -> 0.00 mm
- net /Scheduler/StampClock/C0: track 0.00 -> 40.5 mm
- net /Scheduler/StampClock/S2: track 39.1 -> 0.00 mm
- net /Scheduler/StampClock/S0: track 38.6 -> 0.00 mm
- net /Scheduler/StampClock/S1: track 38.2 -> 0.00 mm
- net ~T_STOP_STB: track 127.5 -> 149.6 mm
- net ~RWD_STB: track 134.0 -> 153.6 mm
- net Net-(Q905-Pad3): track 28.8 -> 47.1 mm
- net Net-(SW981-Pad2): track 43.2 -> 25.6 mm
- net I1: track 138.0 -> 150.5 mm, vias 2 -> 3
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Other:
- outline, holes or cut-outs redrawn
- board text added: "220_R1 (TAPE1 REW) >"
- board text added: "< 220_R2 (TAPE2 REW)"
- board text added: "A"
- board text added: "REV 2"
- board text added: "~F"
- board text removed: "220_R1 (TAPE1 RW) >"
- board text removed: "< 220_R2 (TAPE2 RW)"
- board text removed: "REV 1"
