File: Decoder/Decoder.sch (KiCad schematic (older format))
At the start: 1 part

Commit message: Decoder 1 Rev 1
Parts:
- removed JA4: Conn_02x28_Top_Bottom, symbol Connector_Generic:Conn_02x28_Top_Bottom
- added C11, C12, C13, C14, C17, C19, C24, C25, C26, C5, C6, C7: .1u, Capacitor_THT:C_Disc_D7.0mm_W2.5mm_P5.00mm, symbol Device:C
- added C15, C20, C4, C8, C9: 6V47u, Capacitor_THT:CP_Radial_D6.3mm_P2.50mm, symbol Device:CP
- added C16: .1, Capacitor_THT:C_Disc_D7.0mm_W2.5mm_P5.00mm, symbol Device:C
- added H901, H902, H903, H904: MountingHole, MountingHole:MountingHole_3.2mm_M3, symbol Mechanical:MountingHole
- added J4A1: EdgeTop, Datapoint2200:EdgeConn_28_Pin_Pitch_3.96mm, symbol Connector:Conn_01x28_Male
- added J4B1: EdgeBottom, Datapoint2200:EdgeConn_28_Pin_Pitch_3.96mm, symbol Connector:Conn_01x28_Male
Connections:
- net +12V: now also J4B1.2 (Pin_2)
- net +5V: now also C11.2, C12.2, C13.1, C14.2, C15.1, C16.1, C17.1, C19.1, C20.1, C24.1, C25.1, C26.2, C4.1, C5.2, C6.2, C7.2, C8.1, C9.1, J4B1.1 (Pin_1), J4B1.28 (Pin_28)
- net -12V: now also J4A1.2 (Pin_2)
- net 1.2MHz: now also J4B1.6 (Pin_6)
- net 1.5KC: now also J4A1.13 (Pin_13)
- net 220_R1: now also J4B1.12 (Pin_12)
- net 220_R2: now also J4A1.11 (Pin_11)
- net 7.5CPS: now also J4A1.15 (Pin_15)
- net BEEP: now also J4B1.3 (Pin_3)
- net DECK_1: now also J4A1.12 (Pin_12)
- net DIV64_CLK: now also J4B1.5 (Pin_5)
- net EN_COMP: now also J4B1.9 (Pin_9)
- net GND: now also C11.1, C12.1, C13.2, C14.1, C15.2, C16.2, C17.2, C19.2, C20.2, C24.2, C25.2, C26.1, C4.2, C5.1, C6.1, C7.1, C8.2, C9.2, J4A1.1 (Pin_1), J4A1.28 (Pin_28)
- net INH_MEM: now also J4B1.10 (Pin_10)
- net INT_FACE_CLK: now also J4B1.11 (Pin_11)
- net PHASE_CLK: now also J4A1.4 (Pin_4)
- net PHI1_MEM: now also J4A1.7 (Pin_7)
- net PHI1_REG: now also J4A1.6 (Pin_6)
- net PHI2_MEM: now also J4B1.7 (Pin_7)
- net REWIND: now also J4B1.13 (Pin_13)
- net SPEAKER: now also J4A1.14 (Pin_14)
- net STROBE_1: now also J4A1.9 (Pin_9)
- net STROBE_2: now also J4B1.8 (Pin_8)
- net STROBE_3: now also J4A1.3 (Pin_3)
- net STROBE_4: now also J4A1.8 (Pin_8)
- net ~ADDRESS: now also J4B1.14 (Pin_14)
- net ~BACK_SPACE_STB: now also J4A1.23 (Pin_23)
- net ~COM_1: now also J4B1.25 (Pin_25)
- net ~COM_2: now also J4B1.26 (Pin_26)
- net ~COM_3: now also J4B1.27 (Pin_27)
- net ~COM_4: now also J4B1.23 (Pin_23)
- net ~DECK_1_STB: now also J4B1.16 (Pin_16)
- net ~DECK_2_STB: now also J4B1.18 (Pin_18)
- net ~DIV64_CLK: now also J4A1.5 (Pin_5)
- net ~ENABLE_1: now also J4B1.22 (Pin_22)
- net ~ENABLE_2: now also J4A1.22 (Pin_22)
- net ~I1: now also J4A1.18 (Pin_18)
- net ~I2: now also J4A1.19 (Pin_19)
- net ~I3: now also J4A1.20 (Pin_20)
- net ~I4: now also J4A1.21 (Pin_21)
- net ~POR: now also J4B1.15 (Pin_15)
- net ~READ_BLK_STB: now also J4A1.16 (Pin_16)
- net ~RWD_STB: now also J4A1.26 (Pin_26)
- net ~SENSE_DATA_STB: now also J4B1.19 (Pin_19)
- net ~SENSE_STATUS_STB: now also J4B1.20 (Pin_20)
- net ~SLEW_FWB_STB: now also J4A1.24 (Pin_24)
- net ~SLEW_REV_STB: now also J4A1.25 (Pin_25)
- net ~T1: now also J4A1.10 (Pin_10)
- net ~T_STOP_STB: now also J4A1.27 (Pin_27)
- net ~WRITE_BLK_STB: now also J4B1.17 (Pin_17)
- net ~WRITE_EOF_STB: now also J4A1.17 (Pin_17)
- net ~WRITE_STB: now also J4B1.24 (Pin_24)
- new net ~ADR_STB: J4B1.21 (Pin_21)
Other:
- note added: "3.96mm pitch"

Commit message: Schematics for display & keyboard, adding LEDs to processor PCB
Parts:
- added H907, H908: MountingHole, MountingHole:MountingHole_3.2mm_M3, symbol Mechanical:MountingHole
Connections:
- net ~I1 renamed I1
- net ~I2 renamed I2
- net ~I3 renamed I3
- net ~I4 renamed I4
Other:
- note added: "Edge connector"
- note added: "H"
- note added: "History\nRev 1: Original\nRev 2: Fixed footprints for Z14, Z21. Added WORD_SELECT input.\n\nToDo:\nRevise mounting hole positions to better fit processor board."
- note added: "Recommended connector:\nEDAC 305-056-521-202\n3.56mm row spacing\n-056- if pin count\n-521- is pin type (520 is longer, fatter, pins)\n-202 is mounting style. x02 is 3.25mm (.128") dia holes"
- moved on the sheet: H901, H902, H903, H904
Changed lines of the file:
@@
 encoding utf-8
 Sheet 1 7
-Title "Datapoint 2200 Decoder I"
+Title "Datapoint 2200 Decoder I (A4)"
 Date ""
 Rev "1"
@@
 $EndDescr
 $Sheet
-S 3400 1350 1050 3000
+S 3400 1350 1050 1900
 U 627A4461
 F0 "Scheduler" 50
@@
 $EndSheet
 $Sheet
-S 6050 1350 1150 4400
+S 6050 1350 1150 3600
 U 628221FF
 F0 "IODecoder" 50
@@
 F19 "~WRITE_EOF_STB" O R 7200 2850 50
 F20 "~ENABLE_2" I L 6050 1600 50
-F21 "~I4" I L 6050 2250 50
-F22 "~I3" I L 6050 2100 50
-F23 "~I2" I L 6050 1950 50
-F24 "~I1" I L 6050 1800 50
+F21 "I4" I L 6050 2250 50
+F22 "I3" I L 6050 2100 50
+F23 "I2" I L 6050 1950 50
+F24 "I1" I L 6050 1800 50
 F25 "~ENABLE_1" I L 6050 1450 50
 F26 "~ADDRESS" I L 6050 2450 50
@@
 Z
 Text GLabel 1200 3350 0    50   Output ~ 0
-~I2
+I2
 Text GLabel 1200 3250 0    50   Output ~ 0
-~I1
+I1
 Text GLabel 1200 3450 0    50   Output ~ 0
-~I3
+I3
 Text GLabel 1200 3550 0    50   Output ~ 0
-~I4
+I4
 Text GLabel 1200 3650 0    50   Output ~ 0
 ~ENABLE_2
@@
 PHI2_MEM
 Text Notes 2050 2150 0    50   ~ 0
-K
+H
 Text GLabel 1200 2150 0    50   Input ~ 0
 PHI1_MEM
@@
 ~WRITE_EOF_STB
 Text GLabel 5950 1800 0    50   Input ~ 0
-~I1
+I1
 Text GLabel 5950 1950 0    50   Input ~ 0
-~I2
+I2
 Text GLabel 5950 2100 0    50   Input ~ 0
-~I3
+I3
 Text GLabel 5950 2250 0    50   Input ~ 0
-~I4
+I4
 Text GLabel 5950 1600 0    50   Input ~ 0
 ~ENABLE_2
@@
 L Mechanical:MountingHole H902
 U 1 1 64063A5C
-P 1900 6800
-F 0 "H902" H 2000 6846 50  0000 L CNN
-F 1 "MountingHole" H 2000 6755 50  0000 L CNN
-F 2 "MountingHole:MountingHole_3.2mm_M3" H 1900 6800 50  0001 C CNN
-F 3 "~" H 1900 6800 50  0001 C CNN
-	1    1900 6800
+P 4450 6700
+F 0 "H902" H 4550 6746 50  0000 L CNN
+F 1 "MountingHole" H 4550 6655 50  0000 L CNN
+F 2 "MountingHole:MountingHole_3.2mm_M3" H 4450 6700 50  0001 C CNN
+F 3 "~" H 4450 6700 50  0001 C CNN
+	1    4450 6700
 	1    0    0    -1
 $EndComp
@@
 L Mechanical:MountingHole H903
 U 1 1 64063E0C
-P 1900 7100
-F 0 "H903" H 2000 7146 50  0000 L CNN
-F 1 "MountingHole" H 2000 7055 50  0000 L CNN
-F 2 "MountingHole:MountingHole_3.2mm_M3" H 1900 7100 50  0001 C CNN
-F 3 "~" H 1900 7100 50  0001 C CNN
-	1    1900 7100
+P 4450 7000
+F 0 "H903" H 4550 7046 50  0000 L CNN
+F 1 "MountingHole" H 4550 6955 50  0000 L CNN
+F 2 "MountingHole:MountingHole_3.2mm_M3" H 4450 7000 50  0001 C CNN
+F 3 "~" H 4450 7000 50  0001 C CNN
+	1    4450 7000
 	1    0    0    -1
 $EndComp
@@
 L Mechanical:MountingHole H904
 U 1 1 6406407C
-P 1900 7400
-F 0 "H904" H 2000 7446 50  0000 L CNN
-F 1 "MountingHole" H 2000 7355 50  0000 L CNN
-F 2 "MountingHole:MountingHole_3.2mm_M3" H 1900 7400 50  0001 C CNN
-F 3 "~" H 1900 7400 50  0001 C CNN
-	1    1900 7400
+P 4450 7300
+F 0 "H904" H 4550 7346 50  0000 L CNN
+F 1 "MountingHole" H 4550 7255 50  0000 L CNN
+F 2 "MountingHole:MountingHole_3.2mm_M3" H 4450 7300 50  0001 C CNN
+F 3 "~" H 4450 7300 50  0001 C CNN
+	1    4450 7300
 	1    0    0    -1
 $EndComp
@@
 L Mechanical:MountingHole H901
 U 1 1 640643AA
-P 1900 6500
-F 0 "H901" H 2000 6546 50  0000 L CNN
-F 1 "MountingHole" H 2000 6455 50  0000 L CNN
-F 2 "MountingHole:MountingHole_3.2mm_M3" H 1900 6500 50  0001 C CNN
-F 3 "~" H 1900 6500 50  0001 C CNN
-	1    1900 6500
+P 4450 6400
+F 0 "H901" H 4550 6446 50  0000 L CNN
+F 1 "MountingHole" H 4550 6355 50  0000 L CNN
+F 2 "MountingHole:MountingHole_3.2mm_M3" H 4450 6400 50  0001 C CNN
+F 3 "~" H 4450 6400 50  0001 C CNN
+	1    4450 6400
 	1    0    0    -1
 $EndComp
@@
 Wire Wire Line
 	2300 1550 2050 1550
+Text Notes 600  6250 0    50   ~ 0
+History\nRev 1: Original\nRev 2: Fixed footprints for Z14, Z21. Added WORD_SELECT input.\n\nToDo:\nRevise mounting hole positions to better fit processor board.
+$Comp
+L Mechanical:MountingHole H907
+U 1 1 643EDBD3
+P 5450 6400
+F 0 "H907" H 5550 6446 50  0000 L CNN
+F 1 "MountingHole" H 5550 6355 50  0000 L CNN
+F 2 "MountingHole:MountingHole_3.2mm_M3" H 5450 6400 50  0001 C CNN
+F 3 "~" H 5450 6400 50  0001 C CNN
+	1    5450 6400
+	1    0    0    -1
+$EndComp
+$Comp
+L Mechanical:MountingHole H908
+U 1 1 643EE025
+P 5450 6700
+F 0 "H908" H 5550 6746 50  0000 L CNN
+F 1 "MountingHole" H 5550 6655 50  0000 L CNN
+F 2 "MountingHole:MountingHole_3.2mm_M3" H 5450 6700 50  0001 C CNN
+F 3 "~" H 5450 6700 50  0001 C CNN
+	1    5450 6700
+	1    0    0    -1
+$EndComp
+Text Notes 1000 4950 0    50   ~ 0
+Recommended connector:\nEDAC 305-056-521-202\n3.56mm row spacing\n-056- if pin count\n-521- is pin type (520 is longer, fatter, pins)\n-202 is mounting style. x02 is 3.25mm (.128") dia holes
+Text Notes 1350 1100 0    50   ~ 0
+Edge connector
 $EndSCHEMATC
