File: Decoder/IODecoder.sch (KiCad schematic (older format))
At the start: 25 parts

Commit message: Decoder 1 Rev 1
Parts:
- added unit 7 of Z10
- added unit 7 of Z15
- added unit 7 of Z22
- R11, R12, R13, R14, R15, R16, R17, R18: value 2k2 -> 470; footprint (none) -> Resistor_THT:R_Axial_DIN0207_L6.3mm_D2.5mm_P7.62mm_Horizontal
- R19, R20, R21, R22, R23, R24, R25, R26, R27: footprint (none) -> Resistor_THT:R_Axial_DIN0207_L6.3mm_D2.5mm_P7.62mm_Horizontal
- Z10, Z15, Z22: value 74LS07 -> 7407; footprint (none) -> Package_DIP:DIP-14_W7.62mm_Socket
- Z13: value 74LS04 -> 7404; footprint (none) -> Package_DIP:DIP-14_W7.62mm_Socket
- Z14: renamed from Z17; value 74LS154 -> 74154; footprint (none) -> Package_DIP:DIP-24_W10.16mm_Socket
- Z21: value 74LS154 -> 74154; footprint (none) -> Package_DIP:DIP-24_W10.16mm_Socket
- Z5: value 74LS10 -> 7410; footprint (none) -> Package_DIP:DIP-14_W7.62mm_Socket
- Z8: value 74LS08 -> 7408; footprint (none) -> Package_DIP:DIP-14_W7.62mm_Socket
Connections:
- net +5V: now also Z10.14 (VCC), Z15.14 (VCC), Z22.14 (VCC)
- net GND: now also Z10.7 (GND), Z15.7 (GND), Z22.7 (GND)
- net ~SENSE_STATUS: now reaches Z14.10 (S9), Z15.3
- net ~SENSE_DATA: now reaches Z14.11 (S10), Z15.1
- net ~WRITE: now reaches Z10.13, Z14.13 (S11)
- net ~COM1: now reaches Z10.5, Z14.14 (S12)
- net ~COM2: now reaches Z10.3, Z14.15 (S13)
- net ~COM3: now reaches Z10.1, Z14.16 (S14)
- net ~COM4: now reaches Z10.11, Z14.17 (S15)
- net ~ADR: now reaches Z10.9, Z14.9 (S8)
- net ~T_STOP: now reaches Z15.9, Z21.17 (S15)
- net ~RWD: now reaches Z15.11, Z21.16 (S14)
- net ~SLEW_FWB: now reaches Z21.14 (S12), Z22.13
- net ~SLEW_REV: now reaches Z15.5, Z21.15 (S13)
- net ~BACK_SPACE: now reaches Z21.13 (S11), Z22.1
- net ~WRITE_BLK: now reaches Z21.10 (S9), Z22.11
- net ~READ_BLK: now reaches Z21.9 (S8), Z22.5
- net ~DECK_2: now reaches Z21.8 (S7), Z22.9
- net ~DECK_1: now reaches Z21.7 (S6), Z22.3
- net ~PORT8: now reaches Z21.1 (S0)
- net ~PORT9: now reaches Z21.2 (S1)
- net ~PORT10: now reaches Z21.3 (S2)
- net ~PORT11: now reaches Z21.4 (S3)
- net Z21_5 renamed ~BEEP
- net Z21_6 renamed ~CLICK
- net ~ADD_STB renamed ~ADR_STB
- no-connect marks 12 -> 8
Other:
- note added: "This page decodes the EX xxx commands, effectively the OUT command.\nZ14 decodes ports 0 to 7, Z21 ports 8 to 24. \n~I1~ thru ~I4~ are the inverted bits of the instruction register\nUnused pins on Z21 are unused ports.\nUnused pins on Z14 are the codings for INput ports - decoded elsewhere."
- moved on the sheet: R11, R12, R13, R14, R15, R16, R17, R18, R19, R20, R21, R22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

Commit message: Schematics for display & keyboard, adding LEDs to processor PCB
Parts:
- R11, R12, R13, R14, R15, R16, R17, R18, R19, R20, R21, R22, R23, R24, R25, R26, R27: footprint Resistor_THT:R_Axial_DIN0207_L6.3mm_D2.5mm_P7.62mm_Horizontal -> Resistor_THT:R_Axial_DIN0207_L6.3mm_D2.5mm_P10.16mm_Horizontal
- Z10, Z15, Z22: symbol 74xx:74LS07 -> Datapoint2200:74LCX07
- Z14, Z21: footprint Package_DIP:DIP-24_W10.16mm_Socket -> Package_DIP:DIP-24_W15.24mm_Socket
Connections:
- net ~I1 renamed I1
- net ~I2 renamed I2
- net ~I3 renamed I3
- net ~I4 renamed I4
- net ~PORT10 renamed ~PORT2
- net ~PORT11 renamed ~PORT3
- net ~PORT8 renamed ~PORT0
- net ~PORT9 renamed ~PORT1
Changed lines of the file:
@@
 F 0 "Z14" H 4350 7050 50  0000 C CNN
 F 1 "74154" H 4400 6950 50  0000 C CNN
-F 2 "Package_DIP:DIP-24_W10.16mm_Socket" H 4200 6050 50  0001 C CNN
+F 2 "Package_DIP:DIP-24_W15.24mm_Socket" H 4200 6050 50  0001 C CNN
 F 3 "http://www.ti.com/lit/gpn/sn74LS154" H 4200 6050 50  0001 C CNN
 	1    4200 6050
@@
 $EndComp
 $Comp
-L 74xx:74LS07 Z10
+L Datapoint2200:74LCX07 Z10
 U 4 1 6274B929
 P 6100 4700
@@
 $EndComp
 $Comp
-L 74xx:74LS07 Z15
+L Datapoint2200:74LCX07 Z15
 U 2 1 6274C9C8
 P 6100 5100
@@
 $EndComp
 $Comp
-L 74xx:74LS07 Z15
+L Datapoint2200:74LCX07 Z15
 U 1 1 6274CCAB
 P 6100 5500
@@
 $EndComp
 $Comp
-L 74xx:74LS07 Z10
+L Datapoint2200:74LCX07 Z10
 U 6 1 6274CF1A
 P 6100 5900
@@
 $EndComp
 $Comp
-L 74xx:74LS07 Z10
+L Datapoint2200:74LCX07 Z10
 U 3 1 6274D237
 P 6100 6300
@@
 $EndComp
 $Comp
-L 74xx:74LS07 Z10
+L Datapoint2200:74LCX07 Z10
 U 2 1 6274D4E0
 P 6100 6700
@@
 $EndComp
 $Comp
-L 74xx:74LS07 Z10
+L Datapoint2200:74LCX07 Z10
 U 1 1 6274D789
 P 6100 7100
@@
 $EndComp
 $Comp
-L 74xx:74LS07 Z10
+L Datapoint2200:74LCX07 Z10
 U 5 1 6274DA32
 P 6100 7500
@@
 F 0 "R12" V 6650 7400 50  0000 C CNN
 F 1 "470" V 6750 7400 50  0000 C CNN
-F 2 "Resistor_THT:R_Axial_DIN0207_L6.3mm_D2.5mm_P7.62mm_Horizontal" V 6680 7400 50  0001 C CNN
+F 2 "Resistor_THT:R_Axial_DIN0207_L6.3mm_D2.5mm_P10.16mm_Horizontal" V 6680 7400 50  0001 C CNN
 F 3 "~" H 6750 7400 50  0001 C CNN
 	1    6750 7400
@@
 F 0 "R16" V 6650 7000 50  0000 C CNN
 F 1 "470" V 6750 7000 50  0000 C CNN
-F 2 "Resistor_THT:R_Axial_DIN0207_L6.3mm_D2.5mm_P7.62mm_Horizontal" V 6680 7000 50  0001 C CNN
+F 2 "Resistor_THT:R_Axial_DIN0207_L6.3mm_D2.5mm_P10.16mm_Horizontal" V 6680 7000 50  0001 C CNN
 F 3 "~" H 6750 7000 50  0001 C CNN
 	1    6750 7000
@@
 F 0 "R15" V 6650 6600 50  0000 C CNN
 F 1 "470" V 6750 6600 50  0000 C CNN
-F 2 "Resistor_THT:R_Axial_DIN0207_L6.3mm_D2.5mm_P7.62mm_Horizontal" V 6680 6600 50  0001 C CNN
+F 2 "Resistor_THT:R_Axial_DIN0207_L6.3mm_D2.5mm_P10.16mm_Horizontal" V 6680 6600 50  0001 C CNN
 F 3 "~" H 6750 6600 50  0001 C CNN
 	1    6750 6600
@@
 F 0 "R14" V 6650 6200 50  0000 C CNN
 F 1 "470" V 6750 6200 50  0000 C CNN
-F 2 "Resistor_THT:R_Axial_DIN0207_L6.3mm_D2.5mm_P7.62mm_Horizontal" V 6680 6200 50  0001 C CNN
+F 2 "Resistor_THT:R_Axial_DIN0207_L6.3mm_D2.5mm_P10.16mm_Horizontal" V 6680 6200 50  0001 C CNN
 F 3 "~" H 6750 6200 50  0001 C CNN
 	1    6750 6200
@@
 F 0 "R13" V 6650 5800 50  0000 C CNN
 F 1 "470" V 6750 5800 50  0000 C CNN
-F 2 "Resistor_THT:R_Axial_DIN0207_L6.3mm_D2.5mm_P7.62mm_Horizontal" V 6680 5800 50  0001 C CNN
+F 2 "Resistor_THT:R_Axial_DIN0207_L6.3mm_D2.5mm_P10.16mm_Horizontal" V 6680 5800 50  0001 C CNN
 F 3 "~" H 6750 5800 50  0001 C CNN
 	1    6750 5800
@@
 F 0 "R17" V 6650 5400 50  0000 C CNN
 F 1 "470" V 6750 5400 50  0000 C CNN
-F 2 "Resistor_THT:R_Axial_DIN0207_L6.3mm_D2.5mm_P7.62mm_Horizontal" V 6680 5400 50  0001 C CNN
+F 2 "Resistor_THT:R_Axial_DIN0207_L6.3mm_D2.5mm_P10.16mm_Horizontal" V 6680 5400 50  0001 C CNN
 F 3 "~" H 6750 5400 50  0001 C CNN
 	1    6750 5400
@@
 F 0 "R18" V 6650 5000 50  0000 C CNN
 F 1 "470" V 6750 5000 50  0000 C CNN
-F 2 "Resistor_THT:R_Axial_DIN0207_L6.3mm_D2.5mm_P7.62mm_Horizontal" V 6680 5000 50  0001 C CNN
+F 2 "Resistor_THT:R_Axial_DIN0207_L6.3mm_D2.5mm_P10.16mm_Horizontal" V 6680 5000 50  0001 C CNN
 F 3 "~" H 6750 5000 50  0001 C CNN
 	1    6750 5000
@@
 F 0 "R11" V 6650 4600 50  0000 C CNN
 F 1 "470" V 6750 4600 50  0000 C CNN
-F 2 "Resistor_THT:R_Axial_DIN0207_L6.3mm_D2.5mm_P7.62mm_Horizontal" V 6680 4600 50  0001 C CNN
+F 2 "Resistor_THT:R_Axial_DIN0207_L6.3mm_D2.5mm_P10.16mm_Horizontal" V 6680 4600 50  0001 C CNN
 F 3 "~" H 6750 4600 50  0001 C CNN
 	1    6750 4600
@@
 	6500 4700 6400 4700
 $Comp
-L 74xx:74LS07 Z15
+L Datapoint2200:74LCX07 Z15
 U 4 1 62A26341
 P 6100 4200
@@
 $EndComp
 $Comp
-L 74xx:74LS07 Z15
+L Datapoint2200:74LCX07 Z15
 U 5 1 62A266B1
 P 6100 3800
@@
 $EndComp
 $Comp
-L 74xx:74LS07 Z22
+L Datapoint2200:74LCX07 Z22
 U 6 1 62A2695A
 P 6100 3000
@@
 $EndComp
 $Comp
-L 74xx:74LS07 Z15
+L Datapoint2200:74LCX07 Z15
 U 3 1 62A26CFF
 P 6100 3400
@@
 $EndComp
 $Comp
-L 74xx:74LS07 Z22
+L Datapoint2200:74LCX07 Z22
 U 1 1 62A26FE2
 P 6100 2600
@@
 $EndComp
 $Comp
-L 74xx:74LS07 Z22
+L Datapoint2200:74LCX07 Z22
 U 5 1 62A2728B
 P 6100 2100
@@
 $EndComp
 $Comp
-L 74xx:74LS07 Z22
+L Datapoint2200:74LCX07 Z22
 U 3 1 62A27534
 P 6100 1700
@@
 $EndComp
 $Comp
-L 74xx:74LS07 Z22
+L Datapoint2200:74LCX07 Z22
 U 4 1 62A277DD
 P 6100 1300
@@
 $EndComp
 $Comp
-L 74xx:74LS07 Z22
+L Datapoint2200:74LCX07 Z22
 U 2 1 62A27AFF
 P 6100 900
@@
 F 0 "Z21" H 4350 3000 50  0000 C CNN
 F 1 "74154" H 4400 2900 50  0000 C CNN
-F 2 "Package_DIP:DIP-24_W10.16mm_Socket" H 4200 2000 50  0001 C CNN
+F 2 "Package_DIP:DIP-24_W15.24mm_Socket" H 4200 2000 50  0001 C CNN
 F 3 "http://www.ti.com/lit/gpn/sn74LS154" H 4200 2000 50  0001 C CNN
 	1    4200 2000
@@
 F 0 "R19" V 6650 4100 50  0000 C CNN
 F 1 "2k2" V 6750 4100 50  0000 C CNN
-F 2 "Resistor_THT:R_Axial_DIN0207_L6.3mm_D2.5mm_P7.62mm_Horizontal" V 6680 4100 50  0001 C CNN
+F 2 "Resistor_THT:R_Axial_DIN0207_L6.3mm_D2.5mm_P10.16mm_Horizontal" V 6680 4100 50  0001 C CNN
 F 3 "~" H 6750 4100 50  0001 C CNN
 	1    6750 4100
@@
 F 0 "R20" V 6650 3700 50  0000 C CNN
 F 1 "2k2" V 6750 3700 50  0000 C CNN
-F 2 "Resistor_THT:R_Axial_DIN0207_L6.3mm_D2.5mm_P7.62mm_Horizontal" V 6680 3700 50  0001 C CNN
+F 2 "Resistor_THT:R_Axial_DIN0207_L6.3mm_D2.5mm_P10.16mm_Horizontal" V 6680 3700 50  0001 C CNN
 F 3 "~" H 6750 3700 50  0001 C CNN
 	1    6750 3700
@@
 F 0 "R21" V 6650 3300 50  0000 C CNN
 F 1 "2k2" V 6750 3300 50  0000 C CNN
-F 2 "Resistor_THT:R_Axial_DIN0207_L6.3mm_D2.5mm_P7.62mm_Horizontal" V 6680 3300 50  0001 C CNN
+F 2 "Resistor_THT:R_Axial_DIN0207_L6.3mm_D2.5mm_P10.16mm_Horizontal" V 6680 3300 50  0001 C CNN
 F 3 "~" H 6750 3300 50  0001 C CNN
 	1    6750 3300
@@
 F 0 "R22" V 6650 2900 50  0000 C CNN
 F 1 "2k2" V 6750 2900 50  0000 C CNN
-F 2 "Resistor_THT:R_Axial_DIN0207_L6.3mm_D2.5mm_P7.62mm_Horizontal" V 6680 2900 50  0001 C CNN
+F 2 "Resistor_THT:R_Axial_DIN0207_L6.3mm_D2.5mm_P10.16mm_Horizontal" V 6680 2900 50  0001 C CNN
 F 3 "~" H 6750 2900 50  0001 C CNN
 	1    6750 2900
@@
 F 0 "R23" V 6650 2500 50  0000 C CNN
 F 1 "2k2" V 6750 2500 50  0000 C CNN
-F 2 "Resistor_THT:R_Axial_DIN0207_L6.3mm_D2.5mm_P7.62mm_Horizontal" V 6680 2500 50  0001 C CNN
+F 2 "Resistor_THT:R_Axial_DIN0207_L6.3mm_D2.5mm_P10.16mm_Horizontal" V 6680 2500 50  0001 C CNN
 F 3 "~" H 6750 2500 50  0001 C CNN
 	1    6750 2500
@@
 F 0 "R26" V 6650 2000 50  0000 C CNN
 F 1 "2k2" V 6750 2000 50  0000 C CNN
-F 2 "Resistor_THT:R_Axial_DIN0207_L6.3mm_D2.5mm_P7.62mm_Horizontal" V 6680 2000 50  0001 C CNN
+F 2 "Resistor_THT:R_Axial_DIN0207_L6.3mm_D2.5mm_P10.16mm_Horizontal" V 6680 2000 50  0001 C CNN
 F 3 "~" H 6750 2000 50  0001 C CNN
 	1    6750 2000
@@
 F 0 "R24" V 6650 1600 50  0000 C CNN
 F 1 "2k2" V 6750 1600 50  0000 C CNN
-F 2 "Resistor_THT:R_Axial_DIN0207_L6.3mm_D2.5mm_P7.62mm_Horizontal" V 6680 1600 50  0001 C CNN
+F 2 "Resistor_THT:R_Axial_DIN0207_L6.3mm_D2.5mm_P10.16mm_Horizontal" V 6680 1600 50  0001 C CNN
 F 3 "~" H 6750 1600 50  0001 C CNN
 	1    6750 1600
@@
 F 0 "R27" V 6650 1200 50  0000 C CNN
 F 1 "2k2" V 6750 1200 50  0000 C CNN
-F 2 "Resistor_THT:R_Axial_DIN0207_L6.3mm_D2.5mm_P7.62mm_Horizontal" V 6680 1200 50  0001 C CNN
+F 2 "Resistor_THT:R_Axial_DIN0207_L6.3mm_D2.5mm_P10.16mm_Horizontal" V 6680 1200 50  0001 C CNN
 F 3 "~" H 6750 1200 50  0001 C CNN
 	1    6750 1200
@@
 F 0 "R25" V 6650 800 50  0000 C CNN
 F 1 "2k2" V 6750 800 50  0000 C CNN
-F 2 "Resistor_THT:R_Axial_DIN0207_L6.3mm_D2.5mm_P7.62mm_Horizontal" V 6680 800 50  0001 C CNN
+F 2 "Resistor_THT:R_Axial_DIN0207_L6.3mm_D2.5mm_P10.16mm_Horizontal" V 6680 800 50  0001 C CNN
 F 3 "~" H 6750 800 50  0001 C CNN
 	1    6750 800
@@
 ~ENABLE_2
 Text HLabel 3500 1150 1    50   Input ~ 0
-~I4
+I4
 Text HLabel 3400 1150 1    50   Input ~ 0
-~I3
+I3
 Text HLabel 3300 1150 1    50   Input ~ 0
-~I2
+I2
 Text HLabel 3200 1150 1    50   Input ~ 0
-~I1
+I1
 Text HLabel 3100 1150 1    50   Input ~ 0
 ~ENABLE_1
@@
 F8 "~COM3" I L 1600 9000 50
 F9 "~COM4" I L 1600 9100 50
-F10 "~PORT8" I L 1600 9300 50
-F11 "~PORT9" I L 1600 9400 50
-F12 "~PORT10" I L 1600 9500 50
-F13 "~PORT11" I L 1600 9600 50
+F10 "~PORT0" I L 1600 9300 50
+F11 "~PORT1" I L 1600 9400 50
+F12 "~PORT2" I L 1600 9500 50
+F13 "~PORT3" I L 1600 9600 50
 F14 "~BEEP" I L 1600 9700 50
 F15 "~CLICK" I L 1600 9800 50
@@
 	1500 10200 1600 10200
 Text GLabel 1500 9300 0    50   Input ~ 0
-~PORT8
+~PORT0
 Text GLabel 1500 9400 0    50   Input ~ 0
-~PORT9
+~PORT1
 Text GLabel 1500 9500 0    50   Input ~ 0
-~PORT10
+~PORT2
 Text GLabel 1500 9600 0    50   Input ~ 0
-~PORT11
+~PORT3
 Wire Wire Line
 	1500 9300 1600 9300
@@
 	1600 9800 1500 9800
 Text GLabel 4800 1200 1    50   Output ~ 0
-~PORT8
+~PORT0
 Text GLabel 4900 1200 1    50   Output ~ 0
-~PORT9
+~PORT1
 Text GLabel 5000 1200 1    50   Output ~ 0
-~PORT10
+~PORT2
 Text GLabel 5100 1200 1    50   Output ~ 0
-~PORT11
+~PORT3
 Text GLabel 5600 1650 1    50   Output ~ 0
 ~READ_BLK
