File: Decoder/Scheduler.sch (KiCad schematic (older format))
At the start: 27 parts, among them Q1 2N23694, Q2 2N23694, U8 74LS08, Y1 9.8400MHz

Commit message: Decoder 1 Rev 1
Parts:
- added H905, H906: MountingHole, MountingHole:MountingHole_3.2mm_M3, symbol Mechanical:MountingHole
- added JP901: CLK SRC, Connector_PinHeader_2.54mm:PinHeader_1x03_P2.54mm_Vertical, symbol Jumper:Jumper_3_Open
- added unit 3 of Z11
- added unit 7 of Z12
- added unit 7 of Z13
- added unit 1 of Z13
- added unit 3 of Z16
- added unit 5 of Z17
- added unit 5 of Z19
- added unit 5 of Z3
- added unit 1 of Z3
- added unit 5 of Z6
- added unit 5 of Z7
- added unit 5 of Z8
- C1, C2, C3: footprint (none) -> Capacitor_THT:C_Disc_D7.0mm_W2.5mm_P5.00mm
- L1: value 120uH 74mA -> 120uH 75mA; footprint (none) -> Inductor_THT:L_Axial_L9.5mm_D4.0mm_P12.70mm_Horizontal_Fastron_SMCC
- Q1, Q2: value 2N23694 -> 2N2369A; footprint (none) -> Package_TO_SOT_THT:TO-18-3; symbol Device:Q_NPN_BCE -> Device:Q_NPN_EBC
- R1, R2, R28, R3, R4, R5, R6: footprint (none) -> Resistor_THT:R_Axial_DIN0207_L6.3mm_D2.5mm_P7.62mm_Horizontal
- Y1: footprint (none) -> Crystal:Crystal_HC49-U_Horizontal
- Z11, Z16: value 74LS74 -> 7474; footprint (none) -> Package_DIP:DIP-14_W7.62mm_Socket
- Z12, Z13: value 74LS04 -> 7404; footprint (none) -> Package_DIP:DIP-14_W7.62mm_Socket
- Z15: value 74LS07 -> 7407
- Z17, Z7: value 74LS00 -> 7400; footprint (none) -> Package_DIP:DIP-14_W7.62mm_Socket
- Z18: renamed from Z14; value 74LS93 -> 7493; footprint (none) -> Package_DIP:DIP-14_W7.62mm_Socket
- Z19, Z3, Z6: value 74LS02 -> 7402; footprint (none) -> Package_DIP:DIP-14_W7.62mm_Socket
- Z2: value 74LS90 -> 7490; footprint (none) -> Package_DIP:DIP-14_W7.62mm_Socket
- Z8: renamed from U8; value 74LS08 -> 7408; footprint (none) -> Package_DIP:DIP-14_W7.62mm_Socket
Connections:
- net +5V: now also Z11.2 (D), Z11.3 (C), Z11.14 (VCC), Z12.14 (VCC), Z13.1, Z13.14 (VCC), Z16.14 (VCC), Z17.14 (VCC), Z19.14 (VCC), Z3.14 (VCC), Z3.2, Z3.3, Z6.14 (VCC), Z7.14 (VCC), Z8.14 (VCC)
- net 9.84MHz: now also Q2.3 (C), JP901.1 (A); no longer Q2.2 (C), Z11.11 (C)
- net GND: now also Q2.1 (E), Z11.7 (GND), Z12.7 (GND), Z13.7 (GND), Z16.7 (GND), Z17.7 (GND), Z19.7 (GND), Z3.7 (GND), Z6.7 (GND), Z7.7 (GND), Z8.7 (GND); no longer Q2.3 (E), Z11.2 (D), Z11.3 (C)
- net T1: now also Z12.1
- net T2: no longer Z12.1
- net at C1.1, R1.1, R2.2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: now also Q1.2 (B); no longer Q1.1 (B)
- net at C1.2, C2.1, L1.1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: now also Q1.1 (E); no longer Q1.3 (E)
- net at C3.2, R2.1, R3.2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: now also Q1.3 (C); no longer Q1.2 (C)
- net at C3.1, R3.1, R6.2: now also Q2.2 (B); no longer Q2.1 (B)
- net S0: now reaches Z12.11, Z2.1 (CP1..3), Z2.12 (Q0), Z3.12, Z7.10
- net S2: now reaches Z2.8 (Q2), Z3.5
- net S1: now reaches Z2.9 (Q1), Z3.11
- net DIV64 renamed S3
- new net RP_CLK: JP901.3 (B)
- new net SYS_CLK: JP901.2 (C), Z11.11 (C)
- no-connect marks 3 -> 5
Other:
- note added: "For crystal"
- note added: "Original schematics show Q1, Q2 as 2N23694,\nbut no such transistor exists. Graphics card uses\n2N2369A for the same circuit. The '4' is probably \na transcription error."
- note removed: "Check pinout"

Commit message: Schematics for display & keyboard, adding LEDs to processor PCB
Parts:
- R1, R2, R28, R3, R4, R5, R6: footprint Resistor_THT:R_Axial_DIN0207_L6.3mm_D2.5mm_P7.62mm_Horizontal -> Resistor_THT:R_Axial_DIN0207_L6.3mm_D2.5mm_P10.16mm_Horizontal
- Z15: symbol 74xx:74LS07 -> Datapoint2200:74LCX07
Connections:
- net S0 renamed C0
- net S1 renamed C1
- net S2 renamed C2
- net S3 renamed C3
Other:
- note added: "High on step 0, T1"
- note removed: "High on step 0, T0"
Changed lines of the file:
@@
 Title "Datapoint 2200 Decoder I"
 Date ""
-Rev "1"
+Rev "2"
 Comp ""
 Comment1 "Recreated from original schematics"
@@
 F 0 "R1" V 1600 6250 50  0000 C CNN
 F 1 "1k5" V 1700 6250 50  0000 C CNN
-F 2 "Resistor_THT:R_Axial_DIN0207_L6.3mm_D2.5mm_P7.62mm_Horizontal" V 1630 6250 50  0001 C CNN
+F 2 "Resistor_THT:R_Axial_DIN0207_L6.3mm_D2.5mm_P10.16mm_Horizontal" V 1630 6250 50  0001 C CNN
 F 3 "~" H 1700 6250 50  0001 C CNN
 	1    1700 6250
@@
 F 0 "R2" V 2100 5800 50  0000 C CNN
 F 1 "2k2" V 2200 5800 50  0000 C CNN
-F 2 "Resistor_THT:R_Axial_DIN0207_L6.3mm_D2.5mm_P7.62mm_Horizontal" V 2130 5800 50  0001 C CNN
+F 2 "Resistor_THT:R_Axial_DIN0207_L6.3mm_D2.5mm_P10.16mm_Horizontal" V 2130 5800 50  0001 C CNN
 F 3 "~" H 2200 5800 50  0001 C CNN
 	1    2200 5800
@@
 F 0 "R3" V 2600 5500 50  0000 C CNN
 F 1 "1k" V 2700 5500 50  0000 C CNN
-F 2 "Resistor_THT:R_Axial_DIN0207_L6.3mm_D2.5mm_P7.62mm_Horizontal" V 2630 5500 50  0001 C CNN
+F 2 "Resistor_THT:R_Axial_DIN0207_L6.3mm_D2.5mm_P10.16mm_Horizontal" V 2630 5500 50  0001 C CNN
 F 3 "~" H 2700 5500 50  0001 C CNN
 	1    2700 5500
@@
 F 0 "R4" V 2600 5100 50  0000 C CNN
 F 1 "560" V 2700 5100 50  0000 C CNN
-F 2 "Resistor_THT:R_Axial_DIN0207_L6.3mm_D2.5mm_P7.62mm_Horizontal" V 2630 5100 50  0001 C CNN
+F 2 "Resistor_THT:R_Axial_DIN0207_L6.3mm_D2.5mm_P10.16mm_Horizontal" V 2630 5100 50  0001 C CNN
 F 3 "~" H 2700 5100 50  0001 C CNN
 	1    2700 5100
@@
 F 0 "R5" V 3500 5350 50  0000 C CNN
 F 1 "1k" V 3600 5350 50  0000 C CNN
-F 2 "Resistor_THT:R_Axial_DIN0207_L6.3mm_D2.5mm_P7.62mm_Horizontal" V 3530 5350 50  0001 C CNN
+F 2 "Resistor_THT:R_Axial_DIN0207_L6.3mm_D2.5mm_P10.16mm_Horizontal" V 3530 5350 50  0001 C CNN
 F 3 "~" H 3600 5350 50  0001 C CNN
 	1    3600 5350
@@
 F 0 "R6" V 3050 6150 50  0000 C CNN
 F 1 "1k" V 3150 6150 50  0000 C CNN
-F 2 "Resistor_THT:R_Axial_DIN0207_L6.3mm_D2.5mm_P7.62mm_Horizontal" V 3080 6150 50  0001 C CNN
+F 2 "Resistor_THT:R_Axial_DIN0207_L6.3mm_D2.5mm_P10.16mm_Horizontal" V 3080 6150 50  0001 C CNN
 F 3 "~" H 3150 6150 50  0001 C CNN
 	1    3150 6150
@@
 F 0 "R28" V 9300 7900 50  0000 C CNN
 F 1 "470" V 9400 7900 50  0000 C CNN
-F 2 "Resistor_THT:R_Axial_DIN0207_L6.3mm_D2.5mm_P7.62mm_Horizontal" V 9330 7900 50  0001 C CNN
+F 2 "Resistor_THT:R_Axial_DIN0207_L6.3mm_D2.5mm_P10.16mm_Horizontal" V 9330 7900 50  0001 C CNN
 F 3 "~" H 9400 7900 50  0001 C CNN
 	1    9400 7900
@@
 	12700 8250 12700 8350
 $Comp
-L 74xx:74LS07 Z15
+L Datapoint2200:74LCX07 Z15
 U 6 1 62AE9C50
 P 10700 8850
@@
 High on step 9, T1
 Text Notes 12850 2200 0    50   ~ 0
-High on step 0, T0
+High on step 0, T1
 Text Label 12600 2550 0    50   ~ 0
 STEPS1TO8
@@
 Text GLabel 1200 2550 0    50   Input ~ 0
 PHI1_REG
-Text GLabel 1200 2650 0    50   Input ~ 0
-DIV64_CLK
 Text GLabel 1200 3050 0    50   Input ~ 0
 STROBE_3
 Text GLabel 1200 1850 0    50   Input ~ 0
-S0
+C0
 Text GLabel 1200 1950 0    50   Input ~ 0
-S1
+C1
 Text GLabel 1200 2050 0    50   Input ~ 0
-S2
+C2
 Text GLabel 1200 2150 0    50   Input ~ 0
-S3
+C3
 Text GLabel 1200 3250 0    50   Input ~ 0
 INT_FACE_CLK
@@
 F6 "T2" I L 1300 1650 50
 F7 "T3" I L 1300 1750 50
-F8 "S0" I L 1300 1850 50
-F9 "S1" I L 1300 1950 50
-F10 "S2" I L 1300 2050 50
-F11 "S3" I L 1300 2150 50
+F8 "C0" I L 1300 1850 50
+F9 "C1" I L 1300 1950 50
+F10 "C2" I L 1300 2050 50
+F11 "C3" I L 1300 2150 50
 F12 "INH_MEM" I L 1300 2250 50
 F13 "PHI1_MEM" I L 1300 2350 50
@@
 F21 "STROBE4" I L 1300 3150 50
 F22 "INT_FACE_CLK" I L 1300 3250 50
-F23 "S0B" O R 2400 1650 50
-F24 "S3B" O R 2400 1950 50
-F25 "S1B" O R 2400 1750 50
-F26 "S2B" O R 2400 1850 50
+F23 "C0B" O R 2400 1650 50
+F24 "C3B" O R 2400 1950 50
+F25 "C1B" O R 2400 1750 50
+F26 "C2B" O R 2400 1850 50
 F27 "T3B" O R 2400 1500 50
 F28 "T2B" O R 2400 1400 50
@@
 T3
 Text GLabel 10250 3300 2    50   Output ~ 0
-S0
+C0
 Text GLabel 10350 3850 2    50   Output ~ 0
-S1
+C1
 Text GLabel 10400 3950 2    50   Output ~ 0
-S2
+C2
 Text GLabel 10400 4350 2    50   Output ~ 0
-S3
+C3
 Wire Wire Line
 	3600 5600 3800 5600
@@
 F0 "StampClock" 50
 F1 "StampClock.sch" 50
-F2 "S0" I L 3450 1650 50
-F3 "S1" I L 3450 1750 50
-F4 "S2" I L 3450 1850 50
-F5 "S3" I L 3450 1950 50
+F2 "C0" I L 3450 1650 50
+F3 "C1" I L 3450 1750 50
+F4 "C2" I L 3450 1850 50
+F5 "C3" I L 3450 1950 50
 F6 "T0" I L 3450 1200 50
 F7 "T1" I L 3450 1300 50
@@
 Text Notes 900  8500 0    50   ~ 0
 For crystal
+Text GLabel 1200 2650 0    50   Input ~ 0
+C3
 $EndSCHEMATC
