File: Decoder/Speaker_Tape.sch (KiCad schematic (older format))
At the start: 17 parts

Commit message: Initialise
Other:
- note removed: "Incorrect pinout!!"
Changed lines of the file:
@@
 	5500 3300 5500 3400
 Connection ~ 4600 3300
-Text Notes 5600 2100 0    50   ~ 0
-Incorrect pinout!!
 $Comp
 L 74xx:74LS04 Z13
@@
 	1    0    0    -1
 $EndComp
-Text Notes 9450 4050 0    50   ~ 0
-Incorrect pinout!!
 Wire Wire Line
 	9450 3300 9250 3300

Commit message: Decoder 1 Rev 1
Parts:
- removed Z20, Z4: 75451, Package_DIP:DIP-8_W7.62mm_Socket, symbol DataPoint2200:75451
- added unit 3 of Z1
- added Z20, Z4: 75451, Package_DIP:DIP-8_W7.62mm_Socket, symbol Datapoint2200:75451
- added unit 4 of Z5
- added unit 5 of Z9
- C10: value .01 50V -> .01u 50V; footprint (none) -> Capacitor_THT:C_Disc_D7.0mm_W2.5mm_P5.00mm
- C21, C22, C23: value .001 200V -> .001u 200V; footprint (none) -> Capacitor_THT:C_Disc_D7.0mm_W2.5mm_P5.00mm
- CR1, CR2: footprint (none) -> Diode_THT:D_DO-34_SOD68_P7.62mm_Horizontal
- R10, R7, R8, R9: footprint (none) -> Resistor_THT:R_Axial_DIN0207_L6.3mm_D2.5mm_P7.62mm_Horizontal
- Z1: value 74LS74 -> 7474; footprint (none) -> Package_DIP:DIP-14_W7.62mm_Socket
- Z13: value 74LS04 -> 7404; footprint (none) -> Package_DIP:DIP-14_W7.62mm_Socket
- Z5: value 74LS10 -> 7410; footprint (none) -> Package_DIP:DIP-14_W7.62mm_Socket
- Z8: value 74LS08 -> 7408; footprint (none) -> Package_DIP:DIP-14_W7.62mm_Socket
- Z9: value 74LS00 -> 7400; footprint (none) -> Package_DIP:DIP-14_W7.62mm_Socket
Connections:
- net +5V: now also Z1.14 (VCC), Z20.8 (Vcc), Z4.8 (Vcc), Z5.14 (VCC), Z9.14 (VCC)
- net 220_R1: now also Z20.5
- net 220_R2: now also Z20.3
- net BEEP: now also Z4.1, Z4.2
- net DECK_1: now also Z20.6
- net GND: now also Z1.7 (GND), Z20.4 (GND), Z4.4 (GND), Z5.7 (GND), Z9.7 (GND)
- net REWIND: now also Z20.2, Z20.7
- net SP2: now reaches R8.1
- net SP2: now also Z4.3
- net SP1: now reaches R7.1
- net SP1: now also Z4.5
- net at Z9.11: now also Z4.6, Z4.7
- net at Z13.8: now also Z20.1
- net Z21_5 renamed ~BEEP
- net Z21_6 renamed ~CLICK

Commit message: Schematics for display & keyboard, adding LEDs to processor PCB
Parts:
- R10, R7, R8, R9: footprint Resistor_THT:R_Axial_DIN0207_L6.3mm_D2.5mm_P7.62mm_Horizontal -> Resistor_THT:R_Axial_DIN0207_L6.3mm_D2.5mm_P10.16mm_Horizontal
Changed lines of the file:
@@
 F 0 "R10" V 3000 2550 50  0000 C CNN
 F 1 "10k" V 3100 2550 50  0000 C CNN
-F 2 "Resistor_THT:R_Axial_DIN0207_L6.3mm_D2.5mm_P7.62mm_Horizontal" V 3030 2550 50  0001 C CNN
+F 2 "Resistor_THT:R_Axial_DIN0207_L6.3mm_D2.5mm_P10.16mm_Horizontal" V 3030 2550 50  0001 C CNN
 F 3 "~" H 3100 2550 50  0001 C CNN
 	1    3100 2550
@@
 F 0 "R9" V 2050 2300 50  0000 C CNN
 F 1 "2k2" V 2150 2300 50  0000 C CNN
-F 2 "Resistor_THT:R_Axial_DIN0207_L6.3mm_D2.5mm_P7.62mm_Horizontal" V 2080 2300 50  0001 C CNN
+F 2 "Resistor_THT:R_Axial_DIN0207_L6.3mm_D2.5mm_P10.16mm_Horizontal" V 2080 2300 50  0001 C CNN
 F 3 "~" H 2150 2300 50  0001 C CNN
 	1    2150 2300
@@
 F 0 "R7" V 6350 2500 50  0000 C CNN
 F 1 "5.1" V 6450 2500 50  0000 C CNN
-F 2 "Resistor_THT:R_Axial_DIN0207_L6.3mm_D2.5mm_P7.62mm_Horizontal" V 6380 2500 50  0001 C CNN
+F 2 "Resistor_THT:R_Axial_DIN0207_L6.3mm_D2.5mm_P10.16mm_Horizontal" V 6380 2500 50  0001 C CNN
 F 3 "~" H 6450 2500 50  0001 C CNN
 	1    6450 2500
@@
 F 0 "R8" V 6350 3300 50  0000 C CNN
 F 1 "1.2" V 6450 3300 50  0000 C CNN
-F 2 "Resistor_THT:R_Axial_DIN0207_L6.3mm_D2.5mm_P7.62mm_Horizontal" V 6380 3300 50  0001 C CNN
+F 2 "Resistor_THT:R_Axial_DIN0207_L6.3mm_D2.5mm_P10.16mm_Horizontal" V 6380 3300 50  0001 C CNN
 F 3 "~" H 6450 3300 50  0001 C CNN
 	1    6450 3300
