File: Memory/Matrix.sch (KiCad schematic (older format))
At the start: 32 parts

Commit message: Schematics for display & keyboard, adding LEDs to processor PCB
Connections:
- net COL0: now also Z14.9 (CS2), Z18.9 (CS2), Z23.9 (CS2), Z27.9 (CS2), Z32.9 (CS2), Z36.9 (CS2), Z5.9 (CS2), Z9.9 (CS2); no longer Z2.1 (CS1), Z3.1 (CS1), Z4.1 (CS1), Z5.1 (CS1)
- net COL1: now also Z13.9 (CS2), Z17.9 (CS2), Z22.9 (CS2), Z26.9 (CS2), Z31.9 (CS2), Z35.9 (CS2), Z4.9 (CS2), Z8.9 (CS2); no longer Z6.1 (CS1), Z7.1 (CS1), Z8.1 (CS1), Z9.1 (CS1)
- net COL2: now also Z12.9 (CS2), Z16.9 (CS2), Z21.9 (CS2), Z25.9 (CS2), Z3.9 (CS2), Z30.9 (CS2), Z34.9 (CS2), Z7.9 (CS2); no longer Z11.1 (CS1), Z12.1 (CS1), Z13.1 (CS1), Z14.1 (CS1)
- net COL3: now also Z11.9 (CS2), Z15.9 (CS2), Z2.9 (CS2), Z20.9 (CS2), Z24.9 (CS2), Z29.9 (CS2), Z33.9 (CS2), Z6.9 (CS2); no longer Z15.1 (CS1), Z16.1 (CS1), Z17.1 (CS1), Z18.1 (CS1)
- net INPUT: now also Z30.3 (INPUT)
- net ROW0: now also Z2.1 (CS1), Z3.1 (CS1), Z4.1 (CS1), Z5.1 (CS1); no longer Z14.9 (CS2), Z18.9 (CS2), Z23.9 (CS2), Z27.9 (CS2), Z32.9 (CS2), Z36.9 (CS2), Z5.9 (CS2), Z9.9 (CS2)
- net ROW1: now also Z6.1 (CS1), Z7.1 (CS1), Z8.1 (CS1), Z9.1 (CS1); no longer Z13.9 (CS2), Z17.9 (CS2), Z22.9 (CS2), Z26.9 (CS2), Z31.9 (CS2), Z35.9 (CS2), Z4.9 (CS2), Z8.9 (CS2)
- net ROW2: now also Z11.1 (CS1), Z12.1 (CS1), Z13.1 (CS1), Z14.1 (CS1); no longer Z12.9 (CS2), Z16.9 (CS2), Z21.9 (CS2), Z25.9 (CS2), Z3.9 (CS2), Z30.9 (CS2), Z34.9 (CS2), Z7.9 (CS2)
- net ROW3: now also Z15.1 (CS1), Z16.1 (CS1), Z17.1 (CS1), Z18.1 (CS1); no longer Z11.9 (CS2), Z15.9 (CS2), Z2.9 (CS2), Z20.9 (CS2), Z24.9 (CS2), Z29.9 (CS2), Z33.9 (CS2), Z6.9 (CS2)
- net COL4 renamed ROW4
- net COL5 renamed ROW5
- net COL6 renamed ROW6
- net COL7 renamed ROW7
Changed lines of the file:
@@
 $Descr A3 16535 11693
 encoding utf-8
-Sheet 2 2
+Sheet 3 3
 Title ""
 Date ""
@@
 U 1 1 6433A02B
 P 2100 2750
+AR Path="/6433A02B" Ref="Z5"  Part="1"
+AR Path="/64339692/6433A02B" Ref="Z5"  Part="1"
 F 0 "Z5" H 2250 2900 50  0000 L CNN
 F 1 "1405" H 2200 2800 50  0000 L CNN
@@
 PHI2_MEM
 Text HLabel 1500 1850 1    50   Input ~ 0
+ROW0
+Text HLabel 3400 1850 1    50   Input ~ 0
+ROW1
+Text HLabel 5300 1850 1    50   Input ~ 0
+ROW2
+Text HLabel 7200 1850 1    50   Input ~ 0
+ROW3
+Text HLabel 9100 1850 1    50   Input ~ 0
+ROW4
+Text HLabel 11000 1850 1    50   Input ~ 0
+ROW5
+Text HLabel 12900 1850 1    50   Input ~ 0
+ROW6
+Text HLabel 14800 1900 1    50   Input ~ 0
+ROW7
+Text HLabel 800  2450 0    50   Input ~ 0
 COL0
-Text HLabel 3400 1850 1    50   Input ~ 0
+Text HLabel 800  4100 0    50   Input ~ 0
 COL1
-Text HLabel 5300 1850 1    50   Input ~ 0
+Text HLabel 800  5750 0    50   Input ~ 0
 COL2
-Text HLabel 7200 1850 1    50   Input ~ 0
+Text HLabel 800  7400 0    50   Input ~ 0
 COL3
-Text HLabel 9100 1850 1    50   Input ~ 0
-COL4
-Text HLabel 11000 1850 1    50   Input ~ 0
-COL5
-Text HLabel 12900 1850 1    50   Input ~ 0
-COL6
-Text HLabel 14800 1900 1    50   Input ~ 0
-COL7
-Text HLabel 800  2450 0    50   Input ~ 0
-ROW0
-Text HLabel 800  4100 0    50   Input ~ 0
-ROW1
-Text HLabel 800  5750 0    50   Input ~ 0
-ROW2
-Text HLabel 800  7400 0    50   Input ~ 0
-ROW3
 Text HLabel 900  1850 1    50   Input ~ 0
 INPUT
@@
 U 1 1 6433C923
 P 2100 4400
+AR Path="/6433C923" Ref="Z4"  Part="1"
+AR Path="/64339692/6433C923" Ref="Z4"  Part="1"
 F 0 "Z4" H 2250 4550 50  0000 L CNN
 F 1 "1405" H 2200 4450 50  0000 L CNN
@@
 U 1 1 6433D0DB
 P 2100 6050
+AR Path="/6433D0DB" Ref="Z3"  Part="1"
+AR Path="/64339692/6433D0DB" Ref="Z3"  Part="1"
 F 0 "Z3" H 2250 6200 50  0000 L CNN
 F 1 "1405" H 2200 6100 50  0000 L CNN
@@
 U 1 1 6433D6E5
 P 2100 7700
+AR Path="/6433D6E5" Ref="Z2"  Part="1"
+AR Path="/64339692/6433D6E5" Ref="Z2"  Part="1"
 F 0 "Z2" H 2250 7850 50  0000 L CNN
 F 1 "1405" H 2200 7750 50  0000 L CNN
@@
 U 1 1 6433DCB7
 P 4000 2750
+AR Path="/6433DCB7" Ref="Z9"  Part="1"
+AR Path="/64339692/6433DCB7" Ref="Z9"  Part="1"
 F 0 "Z9" H 4150 2900 50  0000 L CNN
 F 1 "1405" H 4100 2800 50  0000 L CNN
@@
 U 1 1 6433E437
 P 5900 2750
+AR Path="/6433E437" Ref="Z14"  Part="1"
+AR Path="/64339692/6433E437" Ref="Z14"  Part="1"
 F 0 "Z14" H 6050 2900 50  0000 L CNN
 F 1 "1405" H 6000 2800 50  0000 L CNN
@@
 U 1 1 6433E925
 P 7800 2750
+AR Path="/6433E925" Ref="Z18"  Part="1"
+AR Path="/64339692/6433E925" Ref="Z18"  Part="1"
 F 0 "Z18" H 7950 2900 50  0000 L CNN
 F 1 "1405" H 7900 2800 50  0000 L CNN
@@
 U 1 1 6433EDAC
 P 9700 2750
+AR Path="/6433EDAC" Ref="Z23"  Part="1"
+AR Path="/64339692/6433EDAC" Ref="Z23"  Part="1"
 F 0 "Z23" H 9850 2900 50  0000 L CNN
 F 1 "1405" H 9800 2800 50  0000 L CNN
@@
 U 1 1 6433F10A
 P 11600 2750
+AR Path="/6433F10A" Ref="Z27"  Part="1"
+AR Path="/64339692/6433F10A" Ref="Z27"  Part="1"
 F 0 "Z27" H 11750 2900 50  0000 L CNN
 F 1 "1405" H 11700 2800 50  0000 L CNN
@@
 U 1 1 6433F550
 P 13500 2750
+AR Path="/6433F550" Ref="Z32"  Part="1"
+AR Path="/64339692/6433F550" Ref="Z32"  Part="1"
 F 0 "Z32" H 13650 2900 50  0000 L CNN
 F 1 "1405" H 13600 2800 50  0000 L CNN
@@
 U 1 1 6433FB47
 P 15400 2750
+AR Path="/6433FB47" Ref="Z36"  Part="1"
+AR Path="/64339692/6433FB47" Ref="Z36"  Part="1"
 F 0 "Z36" H 15550 2900 50  0000 L CNN
 F 1 "1405" H 15500 2800 50  0000 L CNN
@@
 U 1 1 643400EE
 P 4000 4450
+AR Path="/643400EE" Ref="Z8"  Part="1"
+AR Path="/64339692/643400EE" Ref="Z8"  Part="1"
 F 0 "Z8" H 4150 4600 50  0000 L CNN
 F 1 "1405" H 4100 4500 50  0000 L CNN
@@
 U 1 1 643409F2
 P 5900 4450
+AR Path="/643409F2" Ref="Z13"  Part="1"
+AR Path="/64339692/643409F2" Ref="Z13"  Part="1"
 F 0 "Z13" H 6050 4600 50  0000 L CNN
 F 1 "1405" H 6000 4500 50  0000 L CNN
@@
 U 1 1 64340D3C
 P 7800 4450
+AR Path="/64340D3C" Ref="Z17"  Part="1"
+AR Path="/64339692/64340D3C" Ref="Z17"  Part="1"
 F 0 "Z17" H 7950 4600 50  0000 L CNN
 F 1 "1405" H 7900 4500 50  0000 L CNN
@@
 U 1 1 643410F8
 P 9700 4450
+AR Path="/643410F8" Ref="Z22"  Part="1"
+AR Path="/64339692/643410F8" Ref="Z22"  Part="1"
 F 0 "Z22" H 9850 4600 50  0000 L CNN
 F 1 "1405" H 9800 4500 50  0000 L CNN
@@
 U 1 1 6434153C
 P 11600 4450
+AR Path="/6434153C" Ref="Z26"  Part="1"
+AR Path="/64339692/6434153C" Ref="Z26"  Part="1"
 F 0 "Z26" H 11750 4600 50  0000 L CNN
 F 1 "1405" H 11700 4500 50  0000 L CNN
@@
 U 1 1 643418BA
 P 13500 4450
+AR Path="/643418BA" Ref="Z31"  Part="1"
+AR Path="/64339692/643418BA" Ref="Z31"  Part="1"
 F 0 "Z31" H 13650 4600 50  0000 L CNN
 F 1 "1405" H 13600 4500 50  0000 L CNN
@@
 U 1 1 64341C38
 P 15400 4450
+AR Path="/64341C38" Ref="Z35"  Part="1"
+AR Path="/64339692/64341C38" Ref="Z35"  Part="1"
 F 0 "Z35" H 15550 4600 50  0000 L CNN
 F 1 "1405" H 15500 4500 50  0000 L CNN
@@
 U 1 1 64341F58
 P 15400 6050
+AR Path="/64341F58" Ref="Z34"  Part="1"
+AR Path="/64339692/64341F58" Ref="Z34"  Part="1"
 F 0 "Z34" H 15550 6200 50  0000 L CNN
 F 1 "1405" H 15500 6100 50  0000 L CNN
@@
 U 1 1 643424A4
 P 13500 6050
+AR Path="/643424A4" Ref="Z30"  Part="1"
+AR Path="/64339692/643424A4" Ref="Z30"  Part="1"
 F 0 "Z30" H 13650 6200 50  0000 L CNN
 F 1 "1405" H 13600 6100 50  0000 L CNN
@@
 U 1 1 64342A9B
 P 11600 6050
+AR Path="/64342A9B" Ref="Z25"  Part="1"
+AR Path="/64339692/64342A9B" Ref="Z25"  Part="1"
 F 0 "Z25" H 11750 6200 50  0000 L CNN
 F 1 "1405" H 11700 6100 50  0000 L CNN
@@
 U 1 1 64343742
 P 9700 6050
+AR Path="/64343742" Ref="Z21"  Part="1"
+AR Path="/64339692/64343742" Ref="Z21"  Part="1"
 F 0 "Z21" H 9850 6200 50  0000 L CNN
 F 1 "1405" H 9800 6100 50  0000 L CNN
@@
 U 1 1 64343BC1
 P 7800 6050
+AR Path="/64343BC1" Ref="Z16"  Part="1"
+AR Path="/64339692/64343BC1" Ref="Z16"  Part="1"
 F 0 "Z16" H 7950 6200 50  0000 L CNN
 F 1 "1405" H 7900 6100 50  0000 L CNN
@@
 U 1 1 64344059
 P 5900 6050
+AR Path="/64344059" Ref="Z12"  Part="1"
+AR Path="/64339692/64344059" Ref="Z12"  Part="1"
 F 0 "Z12" H 6050 6200 50  0000 L CNN
 F 1 "1405" H 6000 6100 50  0000 L CNN
@@
 U 1 1 6434463C
 P 4000 6050
+AR Path="/6434463C" Ref="Z7"  Part="1"
+AR Path="/64339692/6434463C" Ref="Z7"  Part="1"
 F 0 "Z7" H 4150 6200 50  0000 L CNN
 F 1 "1405" H 4100 6100 50  0000 L CNN
@@
 U 1 1 64344B4D
 P 4000 7700
+AR Path="/64344B4D" Ref="Z6"  Part="1"
+AR Path="/64339692/64344B4D" Ref="Z6"  Part="1"
 F 0 "Z6" H 4150 7850 50  0000 L CNN
 F 1 "1405" H 4100 7750 50  0000 L CNN
@@
 U 1 1 643451EB
 P 5900 7700
+AR Path="/643451EB" Ref="Z11"  Part="1"
+AR Path="/64339692/643451EB" Ref="Z11"  Part="1"
 F 0 "Z11" H 6050 7850 50  0000 L CNN
 F 1 "1405" H 6000 7750 50  0000 L CNN
@@
 U 1 1 64345683
 P 7800 7700
+AR Path="/64345683" Ref="Z15"  Part="1"
+AR Path="/64339692/64345683" Ref="Z15"  Part="1"
 F 0 "Z15" H 7950 7850 50  0000 L CNN
 F 1 "1405" H 7900 7750 50  0000 L CNN
@@
 U 1 1 64345A3A
 P 9700 7700
+AR Path="/64345A3A" Ref="Z20"  Part="1"
+AR Path="/64339692/64345A3A" Ref="Z20"  Part="1"
 F 0 "Z20" H 9850 7850 50  0000 L CNN
 F 1 "1405" H 9800 7750 50  0000 L CNN
@@
 U 1 1 64345DFB
 P 11600 7700
+AR Path="/64345DFB" Ref="Z24"  Part="1"
+AR Path="/64339692/64345DFB" Ref="Z24"  Part="1"
 F 0 "Z24" H 11750 7850 50  0000 L CNN
 F 1 "1405" H 11700 7750 50  0000 L CNN
@@
 U 1 1 64346206
 P 13500 7700
+AR Path="/64346206" Ref="Z29"  Part="1"
+AR Path="/64339692/64346206" Ref="Z29"  Part="1"
 F 0 "Z29" H 13650 7850 50  0000 L CNN
 F 1 "1405" H 13600 7750 50  0000 L CNN
@@
 U 1 1 6434665D
 P 15400 7700
+AR Path="/6434665D" Ref="Z33"  Part="1"
+AR Path="/64339692/6434665D" Ref="Z33"  Part="1"
 F 0 "Z33" H 15550 7850 50  0000 L CNN
 F 1 "1405" H 15500 7750 50  0000 L CNN
@@
 	13000 5350 12300 5350
 Connection ~ 12300 5350
-Wire Wire Line
-	12300 5350 12300 8600
 Wire Wire Line
 	13000 6450 12700 6450
@@
 	-1   0    0    1
 $EndComp
+Wire Wire Line
+	13000 6950 12300 6950
+Wire Wire Line
+	12300 5350 12300 6950
+Connection ~ 12300 6950
+Wire Wire Line
+	12300 6950 12300 8600
 $EndSCHEMATC
