File: Memory/Memory.kicad_pcb (KiCad board)
At the start: 2 copper layers, 133.3 x 203.2 mm, 88 parts, among them J1 Edge_Bottom, J2 Edge_Top, Q1 2N3725, Q2 2N2219, Q3 2N3726, Q4 2N3726, Q5 2N2219, Q6 2N3725

Commit message: Schematics for display & keyboard, adding LEDs to processor PCB
Parts:
- added D901: COL0, DataPoint_2200:LED_Dialight_597_xxxx_407F_SMT_RA_3mmx2mmx1mm, F.Cu at (171.4, 10.8)
- added D902: COL1, DataPoint_2200:LED_Dialight_597_xxxx_407F_SMT_RA_3mmx2mmx1mm, F.Cu at (171.4, 19.1)
- added D903: COL2, DataPoint_2200:LED_Dialight_597_xxxx_407F_SMT_RA_3mmx2mmx1mm, F.Cu at (171.4, 27.3)
- added D904: COL3, DataPoint_2200:LED_Dialight_597_xxxx_407F_SMT_RA_3mmx2mmx1mm, F.Cu at (171.4, 35.6)
- added D905: PHI1, DataPoint_2200:LED_Dialight_597_xxxx_407F_SMT_RA_3mmx2mmx1mm, F.Cu at (171.4, 162.6)
- added D906: PHI2, DataPoint_2200:LED_Dialight_597_xxxx_407F_SMT_RA_3mmx2mmx1mm, F.Cu at (171.4, 170.8)
- added D907: INPUT, DataPoint_2200:LED_Dialight_597_xxxx_407F_SMT_RA_3mmx2mmx1mm, F.Cu at (171.4, 143.5)
- added D908: WRITE, DataPoint_2200:LED_Dialight_597_xxxx_407F_SMT_RA_3mmx2mmx1mm, F.Cu at (171.4, 132.1)
- added D909: READ, DataPoint_2200:LED_Dialight_597_xxxx_407F_SMT_RA_3mmx2mmx1mm, F.Cu at (171.4, 123.9)
- added D910: OUTPUT, DataPoint_2200:LED_Dialight_597_xxxx_407F_SMT_RA_3mmx2mmx1mm, F.Cu at (171.4, 151.8)
- added D911: PAGE_SEL, DataPoint_2200:LED_Dialight_597_xxxx_407F_SMT_RA_3mmx2mmx1mm, F.Cu at (171.4, 115.6)
- added D912: ROW0, DataPoint_2200:LED_Dialight_597_xxxx_407F_SMT_RA_3mmx2mmx1mm, F.Cu at (171.4, 47.0)
- added D913: ROW1, DataPoint_2200:LED_Dialight_597_xxxx_407F_SMT_RA_3mmx2mmx1mm, F.Cu at (171.4, 55.3)
- added D914: ROW2, DataPoint_2200:LED_Dialight_597_xxxx_407F_SMT_RA_3mmx2mmx1mm, F.Cu at (171.4, 63.5)
- added D915: ROW3, DataPoint_2200:LED_Dialight_597_xxxx_407F_SMT_RA_3mmx2mmx1mm, F.Cu at (171.4, 71.8)
- added D916: ROW4, DataPoint_2200:LED_Dialight_597_xxxx_407F_SMT_RA_3mmx2mmx1mm, F.Cu at (171.4, 80.0)
- added D917: ROW5, DataPoint_2200:LED_Dialight_597_xxxx_407F_SMT_RA_3mmx2mmx1mm, F.Cu at (171.4, 88.3)
- added D918: ROW6, DataPoint_2200:LED_Dialight_597_xxxx_407F_SMT_RA_3mmx2mmx1mm, F.Cu at (171.4, 96.6)
- added D919: ROW7, DataPoint_2200:LED_Dialight_597_xxxx_407F_SMT_RA_3mmx2mmx1mm, F.Cu at (171.4, 104.8)
- added D920: Z5, LED_SMD:LED_0805_2012Metric_Pad1.15x1.40mm_HandSolder, F.Cu at (160.7, 15.2)
- added D921: Z4, LED_SMD:LED_0805_2012Metric_Pad1.15x1.40mm_HandSolder, F.Cu at (138.4, 15.2)
- added D922: Z3, LED_SMD:LED_0805_2012Metric_Pad1.15x1.40mm_HandSolder, F.Cu at (108.0, 15.2)
- added D923: Z2, LED_SMD:LED_0805_2012Metric_Pad1.15x1.40mm_HandSolder, F.Cu at (85.7, 15.2)
- added D924: Z9, LED_SMD:LED_0805_2012Metric_Pad1.15x1.40mm_HandSolder, F.Cu at (160.7, 32.4)
- added D925: Z8, LED_SMD:LED_0805_2012Metric_Pad1.15x1.40mm_HandSolder, F.Cu at (138.4, 32.4)
- added D926: Z7, LED_SMD:LED_0805_2012Metric_Pad1.15x1.40mm_HandSolder, F.Cu at (108.0, 32.4)
- added D927: Z6, LED_SMD:LED_0805_2012Metric_Pad1.15x1.40mm_HandSolder, F.Cu at (85.7, 32.4)
- added D928: Z14, LED_SMD:LED_0805_2012Metric_Pad1.15x1.40mm_HandSolder, F.Cu at (160.7, 49.5)
- added D929: Z13, LED_SMD:LED_0805_2012Metric_Pad1.15x1.40mm_HandSolder, F.Cu at (138.4, 49.5)
- added D930: Z12, LED_SMD:LED_0805_2012Metric_Pad1.15x1.40mm_HandSolder, F.Cu at (108.0, 49.5)
- added D931: Z11, LED_SMD:LED_0805_2012Metric_Pad1.15x1.40mm_HandSolder, F.Cu at (85.7, 49.5)
- added D932: Z18, LED_SMD:LED_0805_2012Metric_Pad1.15x1.40mm_HandSolder, F.Cu at (160.7, 66.7)
- added D933: Z17, LED_SMD:LED_0805_2012Metric_Pad1.15x1.40mm_HandSolder, F.Cu at (138.4, 66.7)
- added D934: Z16, LED_SMD:LED_0805_2012Metric_Pad1.15x1.40mm_HandSolder, F.Cu at (108.0, 66.7)
- added D935: Z15, LED_SMD:LED_0805_2012Metric_Pad1.15x1.40mm_HandSolder, F.Cu at (85.7, 66.7)
- added D936: Z23, LED_SMD:LED_0805_2012Metric_Pad1.15x1.40mm_HandSolder, F.Cu at (160.7, 83.8)
- added D937: Z22, LED_SMD:LED_0805_2012Metric_Pad1.15x1.40mm_HandSolder, F.Cu at (138.4, 83.8)
- added D938: Z21, LED_SMD:LED_0805_2012Metric_Pad1.15x1.40mm_HandSolder, F.Cu at (108.0, 83.8)
- added D939: Z20, LED_SMD:LED_0805_2012Metric_Pad1.15x1.40mm_HandSolder, F.Cu at (85.7, 83.8)
- added D940: Z27, LED_SMD:LED_0805_2012Metric_Pad1.15x1.40mm_HandSolder, F.Cu at (160.7, 101.0)
- added D941: Z26, LED_SMD:LED_0805_2012Metric_Pad1.15x1.40mm_HandSolder, F.Cu at (138.4, 101.0)
- added D942: Z25, LED_SMD:LED_0805_2012Metric_Pad1.15x1.40mm_HandSolder, F.Cu at (108.0, 101.0)
- added D943: Z24, LED_SMD:LED_0805_2012Metric_Pad1.15x1.40mm_HandSolder, F.Cu at (85.7, 101.0)
- added D944: Z32, LED_SMD:LED_0805_2012Metric_Pad1.15x1.40mm_HandSolder, F.Cu at (160.7, 118.1)
- added D945: Z31, LED_SMD:LED_0805_2012Metric_Pad1.15x1.40mm_HandSolder, F.Cu at (138.4, 118.1)
- added D946: Z30, LED_SMD:LED_0805_2012Metric_Pad1.15x1.40mm_HandSolder, F.Cu at (108.0, 118.1)
- added D947: Z29, LED_SMD:LED_0805_2012Metric_Pad1.15x1.40mm_HandSolder, F.Cu at (85.7, 118.1)
- added D948: Z36, LED_SMD:LED_0805_2012Metric_Pad1.15x1.40mm_HandSolder, F.Cu at (160.7, 135.3)
- added D949: Z35, LED_SMD:LED_0805_2012Metric_Pad1.15x1.40mm_HandSolder, F.Cu at (138.4, 135.3)
- added D950: Z34, LED_SMD:LED_0805_2012Metric_Pad1.15x1.40mm_HandSolder, F.Cu at (108.0, 135.3)
- added D951: Z33, LED_SMD:LED_0805_2012Metric_Pad1.15x1.40mm_HandSolder, F.Cu at (85.7, 135.3)
- added H901: MountingHole, MountingHole:MountingHole_3.2mm_M3, F.Cu at (47.6, 17.1)
- added H902: MountingHole, MountingHole:MountingHole_3.2mm_M3, F.Cu at (172.1, 1.91)
- added JP901: PHI1 Driver, Jumper:SolderJumper-2_P1.3mm_Open_RoundedPad1.0x1.5mm, B.Cu at (134.6, 151.1)
- added JP902: ~PHI1, Jumper:SolderJumper-2_P1.3mm_Open_RoundedPad1.0x1.5mm, B.Cu at (137.7, 151.1)
- added JP903: PHI2 Driver, Jumper:SolderJumper-2_P1.3mm_Open_RoundedPad1.0x1.5mm, B.Cu at (89.5, 151.1)
- added JP904: ~PHI2, Jumper:SolderJumper-2_P1.3mm_Open_RoundedPad1.0x1.5mm, B.Cu at (86.5, 151.1)
- added JP906: OUTPUT_MEM, Jumper:SolderJumper-2_P1.3mm_Open_RoundedPad1.0x1.5mm, B.Cu at (102.2, 161.7)
- added JP907: COMPARATOR, Jumper:SolderJumper-2_P1.3mm_Open_RoundedPad1.0x1.5mm, B.Cu at (102.2, 169.1)
- added R901: 470R, Resistor_SMD:R_0805_2012Metric_Pad1.20x1.40mm_HandSolder, B.Cu at (171.4, 10.4)
- added R902: 470R, Resistor_SMD:R_0805_2012Metric_Pad1.20x1.40mm_HandSolder, B.Cu at (171.4, 18.7)
- added R903: 470R, Resistor_SMD:R_0805_2012Metric_Pad1.20x1.40mm_HandSolder, B.Cu at (171.4, 26.9)
- added R904: 470R, Resistor_SMD:R_0805_2012Metric_Pad1.20x1.40mm_HandSolder, B.Cu at (171.4, 35.2)
- added R905: 470R, Resistor_SMD:R_0805_2012Metric_Pad1.20x1.40mm_HandSolder, B.Cu at (171.4, 162.2)
- added R906: 470R, Resistor_SMD:R_0805_2012Metric_Pad1.20x1.40mm_HandSolder, B.Cu at (171.4, 170.4)
- added R907: 470R, Resistor_SMD:R_0805_2012Metric_Pad1.20x1.40mm_HandSolder, B.Cu at (171.4, 147.8)
- added R908: 470R, Resistor_SMD:R_0805_2012Metric_Pad1.20x1.40mm_HandSolder, B.Cu at (172.6, 136.4)
- added R909: 470R, Resistor_SMD:R_0805_2012Metric_Pad1.20x1.40mm_HandSolder, B.Cu at (172.2, 128.1)
- added R910: 470R, Resistor_SMD:R_0805_2012Metric_Pad1.20x1.40mm_HandSolder, B.Cu at (171.4, 156.1)
- added R911: 470R, Resistor_SMD:R_0805_2012Metric_Pad1.20x1.40mm_HandSolder, B.Cu at (172.3, 119.7)
- added R912: 470R, Resistor_SMD:R_0805_2012Metric_Pad1.20x1.40mm_HandSolder, B.Cu at (171.7, 46.6)
- added R913: 470R, Resistor_SMD:R_0805_2012Metric_Pad1.20x1.40mm_HandSolder, B.Cu at (171.4, 54.9)
- added R914: 470R, Resistor_SMD:R_0805_2012Metric_Pad1.20x1.40mm_HandSolder, B.Cu at (171.7, 63.1)
- added R915: 470R, Resistor_SMD:R_0805_2012Metric_Pad1.20x1.40mm_HandSolder, B.Cu at (171.4, 71.4)
- added R916: 470R, Resistor_SMD:R_0805_2012Metric_Pad1.20x1.40mm_HandSolder, B.Cu at (171.4, 79.6)
- added R917: 470R, Resistor_SMD:R_0805_2012Metric_Pad1.20x1.40mm_HandSolder, B.Cu at (171.4, 92.4)
- added R918: 470R, Resistor_SMD:R_0805_2012Metric_Pad1.20x1.40mm_HandSolder, B.Cu at (171.7, 100.6)
- added R919: 470R, Resistor_SMD:R_0805_2012Metric_Pad1.20x1.40mm_HandSolder, B.Cu at (171.4, 109.0)
- added R920: 470R, Resistor_SMD:R_0805_2012Metric_Pad1.20x1.40mm_HandSolder, B.Cu at (99.4, 11.2)
- added R921: 470R, Resistor_SMD:R_0805_2012Metric_Pad1.20x1.40mm_HandSolder, B.Cu at (102.5, 11.2)
- added R922: 470R, Resistor_SMD:R_0805_2012Metric_Pad1.20x1.40mm_HandSolder, B.Cu at (133.0, 11.2)
- added R923: 470R, Resistor_SMD:R_0805_2012Metric_Pad1.20x1.40mm_HandSolder, B.Cu at (155.2, 11.2)
- added U904: 74HCT245, Package_SO:TSSOP-20_4.4x6.5mm_P0.65mm, B.Cu at (143.5, 4.70)
- added U905: 74HCT245, Package_SO:TSSOP-20_4.4x6.5mm_P0.65mm, B.Cu at (69.8, 63.6)
- added U906: 74HCT245, Package_SO:TSSOP-20_4.4x6.5mm_P0.65mm, B.Cu at (165.0, 163.7)
- J1: moved to B.Cu
- J2: moved to F.Cu
- Z1, Z19: value 74LS05 -> 7405
- Z10, Z28: value 74LS42 -> 7442
- Z38: value 74LS03 -> 7403
- moved C49 5.72 mm to (113.7, 176.5)
- moved R27 3.17 mm to (134.6, 157.5)
- moved R18 3.05 mm to (157.6, 152.4)
- moved Z5 1.27 mm to (160.7, 22.2)
- turned J1 to 270 degrees
- turned J2 to 90 degrees
Connections:
- net COL4 renamed ROW4
- net COL5 renamed ROW5
- net COL6 renamed ROW6
- net COL7 renamed ROW7
- net Net-(Z1-Pad11) renamed ~COL1
- net Net-(Z1-Pad13) renamed ~COL2
- net Net-(Z1-Pad5) renamed ~COL3
- net Net-(Z1-Pad9) renamed ~COL0
- net OUTPUT renamed ~OUTPUT
- net PAGE_SELECT renamed ~PAGE_SELECT
- R19 pad 2: ROW1 -> COL1
- R20 pad 2: ROW2 -> COL2
- R21 pad 2: ROW3 -> COL3
- R26 pad 1: PHI2_MEM -> Net-(JP903-Pad1)
- R27 pad 1: PHI1_MEM -> Net-(JP901-Pad1)
- R4 pad 2: ROW0 -> COL0
- R5 pad 1: COL0 -> ROW0
- R6 pad 1: COL1 -> ROW1
- R7 pad 1: COL2 -> ROW2
- R8 pad 1: COL3 -> ROW3
- Z1 pad 10: ROW1 -> COL1
- Z1 pad 12: ROW2 -> COL2
- Z1 pad 14: (no net) -> +5V
- Z1 pad 2: COL1 -> ROW1
- Z1 pad 4: COL0 -> ROW0
- Z1 pad 6: ROW3 -> COL3
- Z1 pad 7: (no net) -> GND
- Z1 pad 8: ROW0 -> COL0
- Z11 pad 1: COL2 -> ROW2
- Z11 pad 9: ROW3 -> COL3
- Z12 pad 1: COL2 -> ROW2
- Z12 pad 9: ROW2 -> COL2
- Z13 pad 1: COL2 -> ROW2
- Z13 pad 9: ROW1 -> COL1
- Z14 pad 1: COL2 -> ROW2
- Z14 pad 9: ROW0 -> COL0
- Z15 pad 1: COL3 -> ROW3
- Z15 pad 9: ROW3 -> COL3
- Z16 pad 1: COL3 -> ROW3
- Z16 pad 9: ROW2 -> COL2
- Z17 pad 1: COL3 -> ROW3
- Z17 pad 9: ROW1 -> COL1
- Z18 pad 1: COL3 -> ROW3
- Z18 pad 9: ROW0 -> COL0
- Z19 pad 10: COL3 -> ROW3
- Z19 pad 14: (no net) -> +5V
- Z19 pad 7: (no net) -> GND
- Z19 pad 8: COL2 -> ROW2
- Z2 pad 1: COL0 -> ROW0
- Z2 pad 9: ROW3 -> COL3
- Z20 pad 9: ROW3 -> COL3
- Z21 pad 9: ROW2 -> COL2
- Z22 pad 9: ROW1 -> COL1
- Z23 pad 9: ROW0 -> COL0
- Z24 pad 9: ROW3 -> COL3
- Z25 pad 9: ROW2 -> COL2
- Z26 pad 9: ROW1 -> COL1
- Z27 pad 9: ROW0 -> COL0
- Z29 pad 9: ROW3 -> COL3
- Z3 pad 1: COL0 -> ROW0
- Z3 pad 9: ROW2 -> COL2
- Z30 pad 3: Net-(Z30-Pad3) -> INPUT
- Z30 pad 9: ROW2 -> COL2
- Z31 pad 9: ROW1 -> COL1
- Z32 pad 9: ROW0 -> COL0
- Z33 pad 9: ROW3 -> COL3
- Z34 pad 9: ROW2 -> COL2
- Z35 pad 9: ROW1 -> COL1
- Z36 pad 9: ROW0 -> COL0
- Z37 pad 1: Net-(Z37-Pad1) -> Net-(JP907-Pad2)
- Z37 pad 10: (no net) -> Net-(Z37-Pad10)
- Z37 pad 11: (no net) -> GND
- Z37 pad 5: (no net) -> GND
- Z37 pad 6: (no net) -> Net-(Z37-Pad6)
- Z37 pad 7: (no net) -> GND
- Z37 pad 8: (no net) -> Net-(Z37-Pad6)
- Z38 pad 1: Net-(Z37-Pad1) -> Net-(JP906-Pad1)
- Z38 pad 10: (no net) -> PHI2
- Z38 pad 11: (no net) -> Net-(Z38-Pad11)
- Z38 pad 12: (no net) -> GND
- Z38 pad 13: (no net) -> GND
- Z38 pad 14: (no net) -> +5V
- Z38 pad 4: (no net) -> PHI1
- Z38 pad 5: (no net) -> PHI1
- Z38 pad 6: (no net) -> Net-(JP902-Pad2)
- Z38 pad 7: (no net) -> GND
- Z38 pad 8: (no net) -> Net-(JP904-Pad2)
- Z38 pad 9: (no net) -> PHI2
- Z4 pad 1: COL0 -> ROW0
- Z4 pad 9: ROW1 -> COL1
- Z5 pad 1: COL0 -> ROW0
- Z5 pad 9: ROW0 -> COL0
- Z6 pad 1: COL1 -> ROW1
- Z6 pad 9: ROW3 -> COL3
- Z7 pad 1: COL1 -> ROW1
- Z7 pad 9: ROW2 -> COL2
- Z8 pad 1: COL1 -> ROW1
- Z8 pad 9: ROW1 -> COL1
- Z9 pad 1: COL1 -> ROW1
- Z9 pad 9: ROW0 -> COL0
Routing:
- net +5V: track 0.00 -> 1016.1 mm, vias 0 -> 8
- net -5V: track 0.00 -> 920.6 mm, vias 0 -> 1
- net INPUT: track 0.00 -> 857.3 mm, vias 0 -> 38
- net WRITE_~RECIRCULATE: track 0.00 -> 804.9 mm, vias 0 -> 38
- net OUTPUT_MEM: track 0.00 -> 781.9 mm, vias 0 -> 36
- net READ: track 0.00 -> 756.1 mm, vias 0 -> 39
- net PHI2_MEM: track 0.00 -> 642.2 mm, vias 0 -> 4
- net PHI1_MEM: track 0.00 -> 638.1 mm, vias 0 -> 4
- net ~PAGE_SELECT: track 0.00 -> 318.8 mm, vias 0 -> 3
- net COL1: track 0.00 -> 316.0 mm, vias 0 -> 11
- net COL0: track 0.00 -> 314.2 mm, vias 0 -> 10
- net COL3: track 0.00 -> 281.2 mm, vias 0 -> 12
- net COL2: track 0.00 -> 277.7 mm, vias 0 -> 12
- net R7: track 0.00 -> 193.8 mm, vias 0 -> 2
- net ~C3: track 0.00 -> 177.1 mm, vias 0 -> 8
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- added copper zone on B.Cu, net +5V
- added copper zone on F.Cu, net GND
Other:
- board size 133.3 x 203.2 mm -> 133.3 x 201.3 mm
- net class Power added: clearance 0.2, trace_width 0.4, via_dia 0.8, via_drill 0.4
- board text added: "+12V"
- board text added: "+5V"
- board text added: "-12V"
- board text added: "-5V"
- board text added: "1"
- board text added: "10"
- board text added: "< ~OUTPUT"
- board text added: "> INPUT"
- board text added: "> P10"
- board text added: "> P6"
- board text added: "> P7"
- board text added: "> P8"
- board text added: "> P9"
- board text added: "> PHI1"
- board text added: "> PHI2"
- board text added: "> READ"
- board text added: "> WR/~RECIRC"
- board text added: "> ~PAGE_SEL"
- board text added: "A"
- board text added: "A11 to A14"
- board text added: "BCD TO DECIMAL"
- board text added: "COLUMN 0"
- board text added: "COLUMN 1"
- board text added: "COLUMN 2"
- board text added: "COLUMN 3"
- board text added: "COLUMN DECODE"
- board text added: "DUAL COMP- ARATORS"
- board text added: "GND"
- board text added: "HEX INVERTERS OC"
- board text added: "L"
- board text added: "OUTPUT BUFFER"
- board text added: "OUTPUT LOGIC"
- board text added: "Output source"
- board text added: "PHI1 DRIVER"
- board text added: "PHI1 source for ICs !JP902 is inverted!"
- board text added: "PHI2 DRIVER"
- board text added: "PHI2 source for ICs !JP904 is inverted!"
- board text added: "QUAD 2-INPUT NAND OC"
- board text added: "REV 1"
- board text added: "ROW 0"
- board text added: "ROW 1"
- board text added: "ROW 2"
- board text added: "ROW 3"
- board text added: "ROW 4"
- board text added: "ROW 5"
- board text added: "ROW 6"
- board text added: "ROW 7"
- board text added: "ROW DECODE"
- board text added: "SMT ICs are TSSOP footprint. Right-angle LEDs are Dialight 597_xxx_407F where xxx is colour code. Other LEDs are 0805. SMT resistors are 470ohm, 0805 package. SMT ICs are TSSOP. Solder link options will need to be configured before use. Some solder link options may cause permanent damage! Visit github.com/Bread80/Datapoint2200 for full details."
- board text added: "Serial Memory for Datapoint 2200 (recreation) © Mike Sutton, 2023 - bread80.com"
- board text added: "WARNINGS: NOT compatible with original Datapoint - verify pinouts etc before using with one. NOT engineered for real Intel 1405 ICs - power traces will need beefing up for such use."
