File: Memory/Memory.sch (KiCad schematic (older format))
At the start: 56 parts, among them J1 Edge_Bottom, J2 Edge_Top, Q1 2N3725, Q2 2N2219, Q3 2N3726, Q4 2N3726, Q5 2N2219, Q6 2N3725

Commit message: Schematics for display & keyboard, adding LEDs to processor PCB
Parts:
- added H901, H902: MountingHole, MountingHole:MountingHole_3.2mm_M3, symbol Mechanical:MountingHole
- added JP901: PHI1 Driver, Jumper:SolderJumper-2_P1.3mm_Open_RoundedPad1.0x1.5mm, symbol Device:Jumper_NO_Small
- added JP902: ~PHI1, Jumper:SolderJumper-2_P1.3mm_Open_RoundedPad1.0x1.5mm, symbol Device:Jumper_NO_Small
- added JP903: PHI2 Driver, Jumper:SolderJumper-2_P1.3mm_Open_RoundedPad1.0x1.5mm, symbol Device:Jumper_NO_Small
- added JP904: ~PHI2, Jumper:SolderJumper-2_P1.3mm_Open_RoundedPad1.0x1.5mm, symbol Device:Jumper_NO_Small
- added JP906: OUTPUT_MEM, Jumper:SolderJumper-2_P1.3mm_Open_RoundedPad1.0x1.5mm, symbol Device:Jumper_NO_Small
- added JP907: COMPARATOR, Jumper:SolderJumper-2_P1.3mm_Open_RoundedPad1.0x1.5mm, symbol Device:Jumper_NO_Small
- added unit 7 of Z1
- added unit 7 of Z19
- added unit 3 of Z37
- added unit 2 of Z37
- added unit 2 of Z38
- added unit 3 of Z38
- added unit 4 of Z38
- added unit 5 of Z38
- C3, C39, C41, C42, C43, C45, C46, C47, C48, C6: footprint Capacitor_THT:C_Disc_D4.7mm_W2.5mm_P5.00mm -> Capacitor_THT:C_Disc_D7.0mm_W2.5mm_P5.00mm
- Z1, Z19: value 74LS05 -> 7405
- Z10, Z28: value 74LS42 -> 7442
- Z38: value 74LS03 -> 7403
Connections:
- net +5V: now also Z1.14 (VCC), Z19.14 (VCC), Z38.14 (VCC)
- net COL0: now also R4.2, Z1.8; no longer R5.1, Z1.4
- net COL1: now also R19.2, Z1.10; no longer R6.1, Z1.2
- net COL2: now also R20.2, Z1.12; no longer R7.1, Z19.8
- net COL3: now also R21.2, Z1.6; no longer R8.1, Z19.10
- net GND: now also Z1.7 (GND), Z19.7 (GND), Z37.11 (GND), Z37.5 (+), Z37.7 (V-), Z38.12, Z38.13, Z38.7 (GND)
- net OUTPUT_MEM: now also JP906.2
- net PHI1: now also Z38.4, Z38.5
- net PHI1_MEM: now also JP901.2, JP902.1; no longer R27.1
- net PHI2: now also Z38.10, Z38.9
- net PHI2_MEM: now also JP903.2, JP904.1; no longer R26.1
- net ROW0: now also R5.1, Z1.4; no longer R4.2, Z1.8
- net ROW1: now also R6.1, Z1.2; no longer R19.2, Z1.10
- net ROW2: now also R7.1, Z19.8; no longer R20.2, Z1.12
- net ROW3: now also R8.1, Z19.10; no longer R21.2, Z1.6
- net ~COL0: now reaches Z1.9, Z10.1 (0)
- net ~COL1: now reaches Z1.11, Z10.2 (1)
- net ~COL2: now reaches Z1.13, Z10.3 (2)
- net ~COL3: now reaches Z1.5, Z10.4 (3)
- net at Z37.1: now also JP907.2; no longer Z38.1
- net COL4 renamed ROW4
- net COL5 renamed ROW5
- net COL6 renamed ROW6
- net COL7 renamed ROW7
- net OUTPUT renamed ~OUTPUT
- net PAGE_SELECT renamed ~PAGE_SELECT
- new net: JP903.1, R26.1
- new net: JP901.1, R27.1
- new net: JP906.1, JP907.1, Z38.1
- new net: JP902.2, Z38.6
- new net: JP904.2, Z38.8
- new net: Z37.6 (-), Z37.8
- no-connect marks 8 -> 10
Other:
- note added: "Jumper options:\nPHI1_MEM and PHI2_MEM can each be jumpered to:\n* The output of the driver circuit.\n* The output of the inverted (i.e. buffered) PHIn signal.\nThe latter may be useful if emulating the original memory with individual \nuCs, i.e. one uC per 1405, where it will help with fan-out.\n\nOUTPUT_MEM\n* The original comparator circuit.\n* The original OUTPUT_MEM.\n* The inverted OUTPUT_M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"
- note added: "Revision history\n----------------\nREV 1: Initial version\nREV 2: Improved silkscreen for \njumper options and capacitor values"
- moved on the sheet: C1, C3, Q1, Q2, Q3, R1, R16, R18, R2, R22, R27, R28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
