File: Processor/ALU.sch (KiCad schematic (older format))
At the start: 32 parts, among them U105 74LS06

Commit message: Decoder 1 Rev 1
Connections:
- net W renamed MEM_RW
Changed lines of the file:
@@
 ~IR3
 Text HLabel 7350 7800 0    50   Input ~ 0
-W
+MEM_RW
 Wire Bus Line
 	9200 5750 2700 5750

Commit message: Schematics for display & keyboard, adding LEDs to processor PCB
Parts:
- R18, R20, R21, R22, R23, R24, R61: footprint (none) -> Resistor_THT:R_Axial_DIN0207_L6.3mm_D2.5mm_P10.16mm_Horizontal
- Z1, Z56, Z72, Z73, Z78: value 74LS04 -> 7404; footprint (none) -> Package_DIP:DIP-14_W7.62mm_Socket
- Z105: renamed from U105; value 74LS06 -> 7406; footprint (none) -> Package_DIP:DIP-14_W7.62mm_Socket; symbol 74xx:74LS06 -> Datapoint2200:74LS06
- Z106: value 74LS74 -> 7474; footprint (none) -> Package_DIP:DIP-14_W7.62mm_Socket
- Z107, Z2, Z35, Z57, Z92: value 74LS03 -> 7403; footprint (none) -> Package_DIP:DIP-14_W7.62mm_Socket; symbol 74xx:74LS03 -> Datapoint2200:74LS03
- Z16: renamed from UZ16; value 74LS20 -> 7420; footprint (none) -> Package_DIP:DIP-14_W7.62mm_Socket
- Z17, Z37, Z58: value 74LS00 -> 7400; footprint (none) -> Package_DIP:DIP-14_W7.62mm_Socket
- Z18, Z36, Z77, Z93: value 74LS10 -> 7410; footprint (none) -> Package_DIP:DIP-14_W7.62mm_Socket
- Z53, Z75: value 74LS02 -> 7402; footprint (none) -> Package_DIP:DIP-14_W7.62mm_Socket
- Z74: value 74LS08 -> 7408; footprint (none) -> Package_DIP:DIP-14_W7.62mm_Socket
- Z76: value 74LS30 -> 7430; footprint (none) -> Package_DIP:DIP-14_W7.62mm_Socket
- Z94: value 74LS42 -> 7442; footprint (none) -> Package_DIP:DIP-16_W7.62mm_Socket
Connections:
- net AW: now also Z74.10
- net MEM_RW: no longer Z74.10
- net RA_DATA_OUT: now also Z107.12
- net ~OPCODE_SHIFT: no longer Z107.12
- net ~ADDER_OUT: now reaches Z17.8, Z36.11
- net ADDITION: now reaches Z57.9, Z75.8, Z93.12
- net SUBTRACTION: now reaches Z57.12, Z75.9, Z93.8
- net ~ADDER_CARRY_OUT: now reaches R21.1, Z57.11, Z57.8, Z92.12
Other:
- note added: "ADDER"
- note added: "ALU OPERATION"
- note added: "ALU OUT SELECT"
- note added: "CARRY CLEAR"
- note added: "CARRY CLOCK"
- note added: "CARRY IN SELECT"
- note added: "SHIFT CONTROL"
- note added: "~A0_OUT"
- note added: "~ADC"
- note added: "~ADD"
- note added: "~AND"
- note added: "~CP"
- note added: "~OR"
- note added: "~SBC"
- note added: "~SUB"
- note added: "~XOR"
- note removed: "ADC"
- note removed: "ADD"
- note removed: "AND"
- note removed: "CP"
- note removed: "OR"
- note removed: "SBC"
- note removed: "SUB"
- note removed: "XOR"
- moved on the sheet: R18, R20, R21, R22, R23, R24, R61, Z106B, Z16B, Z17A, Z17B, Z17C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
