File: Processor/ARegister.sch (KiCad schematic (older format))
At the start: 23 parts

Commit message: Schematics for display & keyboard, adding LEDs to processor PCB
Parts:
- R1, R10, R11, R12, R13, R14, R15, R16, R2, R3, R4, R5, R6, R7, R8, R9: footprint (none) -> Resistor_THT:R_Axial_DIN0207_L6.3mm_D2.5mm_P10.16mm_Horizontal
- Z104, Z105: value 74LS06 -> 7406; footprint (none) -> Package_DIP:DIP-14_W7.62mm_Socket; symbol 74xx:74LS06 -> Datapoint2200:74LS06
- Z107: value 74LS03 -> 7403; footprint (none) -> Package_DIP:DIP-14_W7.62mm_Socket; symbol 74xx:74LS03 -> Datapoint2200:74LS03
- Z72: renamed from Z74; value 74LS04 -> 7404; footprint (none) -> Package_DIP:DIP-14_W7.62mm_Socket
- Z73: value 74LS04 -> 7404; footprint (none) -> Package_DIP:DIP-14_W7.62mm_Socket
- Z90, Z91: value 74LS95 -> 7495; footprint (none) -> Package_DIP:DIP-14_W7.62mm_Socket
Connections:
- net +5V: no longer R10.2, R7.2, Z105.10
- net RA_DATA_OUT: now also Z105.13; no longer Z105.11
- net RA4: now reaches Z104.13, Z90.10 (Q3), Z91.1 (Ds)
- net RA5: now reaches Z104.11, Z90.11 (Q2)
- net RA6: now reaches Z104.9, Z90.12 (Q1)
- net RA7: now reaches Z104.1, Z90.13 (Q0)
- net RA1: now reaches Z105.11, Z91.11 (Q2)
- net RA2: now reaches Z105.9, Z91.12 (Q1)
- net RA3: now reaches Z105.1, Z91.13 (Q0)
- net A0_IN renamed AIN0
- net A0_OUT renamed ~A0_OUT
- net ~A0_OUT: now also Z105.12; no longer Z105.10
- net A1_IN renamed AIN1
- net A2_IN renamed AIN2
- net A2_OUT renamed AOUT2
- net A3_IN renamed AIN3
- net A3_OUT renamed AOUT3
- net A4_IN renamed AIN4
- net A4_OUT renamed AOUT4
- net A5_IN renamed AIN5
- net A5_OUT renamed AOUT5
- net A6_IN renamed AIN6
- net A6_OUT renamed AOUT6
- net A7_IN renamed AIN7
- net A7_OUT renamed ~A7_OUT
- new net AOUT1: R10.2, R7.2, Z105.10
Other:
- note added: "A REGISTER"
- note added: "INPUT BUS"
- note added: "OUTPUT BUS"
- note removed: "P5A-16"
- moved on the sheet: R1, R10, R11, R12, R13, R14, R15, R16, R2, R3, R4, R5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
