File: Processor/AddrRegStackControl.sch (KiCad schematic (older format))
At the start: 23 parts, among them U117 74LS40, U14 74LS40

Commit message: Decoder 1 Rev 1
Connections:
- net AA renamed ~MEM_INDIRECT
- net MEM_RD_OR_WR renamed IMM_RD_OR_WR
- net W renamed MEM_RW
- net ~MEM.RD renamed ~IMM_RD
- net ~MEM.WR renamed ~IMM_WR
- net ~MEM_RD_OR_WR renamed ~IMM_RD_OR_WR
Changed lines of the file:
@@
 $Descr A4 11693 8268
 encoding utf-8
-Sheet 8 12
+Sheet 12 12
 Title ""
 Date ""
@@
 	700  3450 600  3450
 Text HLabel 1000 3950 0    50   Input ~ 0
-W
+MEM_RW
 $Comp
 L 74xx:74LS00 Z12
@@
 $EndComp
 Text HLabel 600  5350 1    50   Input ~ 0
-~MEM.RD
+~IMM_RD
 Text HLabel 600  5550 3    50   Input ~ 0
-~MEM.WR
+~IMM_WR
 $Comp
 L 74xx:74LS10 Z13
@@
 	1950 3200 1950 3850
 Text Label 2000 7050 2    50   ~ 0
-~MEM_RD_OR_WR
+~IMM_RD_OR_WR
 Text Label 2100 5450 0    50   ~ 0
-MEM_RD_OR_WR
+IMM_RD_OR_WR
 Wire Wire Line
 	1850 2200 1850 3550
@@
 	6650 5900 6550 5900
 Text HLabel 6650 6250 3    50   Output ~ 0
-AA
+~MEM_INDIRECT
 Wire Wire Line
 	5850 6000 5950 6000
@@
 	3700 6950 4400 6950
 Wire Wire Line
-	2700 1350 2700 1550
-Wire Wire Line
 	3200 1650 2700 1650
 Wire Wire Line
@@
 	500  3650 500  7200
 Connection ~ 2200 4250
-Connection ~ 2700 1550
 Connection ~ 2700 1650
 Wire Wire Line

Commit message: Schematics for display & keyboard, adding LEDs to processor PCB
Parts:
- R49, R50, R51, R54: footprint (none) -> Resistor_THT:R_Axial_DIN0207_L6.3mm_D2.5mm_P10.16mm_Horizontal
- Z10: value 74LS30 -> 7430; footprint (none) -> Package_DIP:DIP-14_W7.62mm_Socket
- Z102, Z30, Z49: value 74LS04 -> 7404; footprint (none) -> Package_DIP:DIP-14_W7.62mm_Socket
- Z103, Z29, Z89: value 74LS03 -> 7403; footprint (none) -> Package_DIP:DIP-14_W7.62mm_Socket; symbol 74xx:74LS03 -> Datapoint2200:74LS03
- Z11, Z13, Z33: value 74LS10 -> 7410; footprint (none) -> Package_DIP:DIP-14_W7.62mm_Socket
- Z116, Z9: value 74LS08 -> 7408; footprint (none) -> Package_DIP:DIP-14_W7.62mm_Socket
- Z117: renamed from U117; value 74LS40 -> 7440; footprint (none) -> Package_DIP:DIP-14_W7.62mm_Socket
- Z12, Z68, Z88: value 74LS00 -> 7400; footprint (none) -> Package_DIP:DIP-14_W7.62mm_Socket
- Z14: renamed from U14; value 74LS40 -> 7440; footprint (none) -> Package_DIP:DIP-14_W7.62mm_Socket
- Z48: value 74LS05 -> 7405; footprint (none) -> Package_DIP:DIP-14_W7.62mm_Socket
- Z70: value 74LS74 -> 7474; footprint (none) -> Package_DIP:DIP-14_W7.62mm_Socket
Connections:
- net AW: now also Z13.13, Z33.2
- net STROBE_2: no longer Z33.2
- net STROBE_4: no longer Z13.13
- net at Z10.5, Z12.11: no longer Z10.6, Z12.8
- net DO_JUMP_CALL_OR_RETURN renamed FLAG_MATCH
- net IMM_RD_OR_WR renamed IND_RD_OR_WR
- net ~IMM_RD renamed ~IND_RD
- net ~IMM_RD_OR_WR renamed ~IND_RD_OR_WR
- net ~IMM_WR renamed ~IND_WR
- net ~JUMP_CALL_FLAG renamed ~JUMP_CALL_TAKE
- net ~RST_JUMP_CALL_FLAG renamed ~EXECUTE_DONE
- new net: Z10.6, Z12.8
Other:
- note added: "A:\nLow to inhibit \nimmediate data?"
- note added: "INDIRECT READ OR\nWRITE CONTROL"
- note added: "PROGRAM COUNTER\nCOUNT ENABLE"
- note added: "Read from or write to (HL)"
- note added: "STACK CONTROL"
- note removed: "Stack Control"
- moved on the sheet: R49, R50, R51, R54, Z102B, Z102C, Z102F, Z10A, Z116B, Z116C, Z117A, Z11A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
