File: Processor/AddressReg.sch (KiCad schematic (older format))
At the start: 19 parts

Commit message: Schematics for display & keyboard, adding LEDs to processor PCB
Parts:
- C55: value .001 -> .001 1kV; footprint (none) -> Capacitor_THT:C_Disc_D7.0mm_W2.5mm_P5.00mm
- R48: footprint (none) -> Resistor_THT:R_Axial_DIN0207_L6.3mm_D2.5mm_P10.16mm_Horizontal
- TP2: footprint (none) -> TestPoint:TestPoint_THTPad_1.5x1.5mm_Drill0.7mm
- Z109, Z110, Z111, Z112: value 74LS193 -> 74193; footprint (none) -> Package_DIP:DIP-16_W7.62mm_Socket
- Z113, Z64, Z65, Z80, Z81, Z84, Z85: value 74LS153 -> 74153; footprint (none) -> Package_DIP:DIP-16_W7.62mm_Socket
- Z117: value 74LS40 -> 7440; footprint (none) -> Package_DIP:DIP-14_W7.62mm_Socket
- Z33: value 74LS10 -> 7410; footprint (none) -> Package_DIP:DIP-14_W7.62mm_Socket
- Z63: value 74HC164 -> 74164; footprint (none) -> Package_DIP:DIP-14_W7.62mm_Socket
- Z67: renamed from Z64; value 74HC164 -> 74164; footprint (none) -> Package_DIP:DIP-14_W7.62mm_Socket
- Z86: value 74LS00 -> 7400; footprint (none) -> Package_DIP:DIP-14_W7.62mm_Socket
Connections:
- net JUMP_CALL_FLAG renamed JUMP_CALL_TAKE
- net V renamed TEMP_ADDR.WR
Other:
- note added: "(to memory cards)"
- note added: "ADDRESS MULTIPLEXERS"
- note added: "ADDRESS REGISTER"
- note added: "In a jump or call instruction the immediate\naddress word is read into the temp register\nbefore being copied to the address\nregister."
- note added: "MEMORY CHIP \nSELECT"
- note added: "MULTIPLEX SELECT"
- note added: "Multiplexers select the source of data to be \nloaded into the Address Register.\nData can be loaded from the stack, the HL \nregisters or the Temp Address Register."
- note added: "Stores either Program Counter(P) or\nvalue from HL registers.\nZ109 to Z112 also act as counters for P."
- note added: "TEMP\nADDRESS\nREGISTER"
- note removed: "Address Register"
- note removed: "Memory IC select"
- note removed: "Temp\nAddress\nRegister"
