File: Processor/Flags.sch (KiCad schematic (older format))
At the start: 15 parts, among them U34 74LS74

Commit message: Decoder 1 Rev 1
Connections:
- net W renamed MEM_RW
Changed lines of the file:
@@
 Connection ~ 2500 2900
 Text HLabel 800  750  0    50   Input ~ 0
-W
+MEM_RW
 Wire Wire Line
 	2700 4050 2800 4050

Commit message: Schematics for display & keyboard, adding LEDs to processor PCB
Parts:
- R34: footprint (none) -> Resistor_THT:R_Axial_DIN0207_L6.3mm_D2.5mm_P10.16mm_Horizontal
- Z1, Z72: value 74LS04 -> 7404; footprint (none) -> Package_DIP:DIP-14_W7.62mm_Socket
- Z15: value 74LS151 -> 74151; footprint (none) -> Package_DIP:DIP-16_W7.62mm_Socket
- Z2, Z35: value 74LS03 -> 7403; footprint (none) -> Package_DIP:DIP-14_W7.62mm_Socket; symbol 74xx:74LS03 -> Datapoint2200:74LS03
- Z27: value 74LS08 -> 7408; footprint (none) -> Package_DIP:DIP-14_W7.62mm_Socket
- Z31, Z34: value 74LS74 -> 7474; footprint (none) -> Package_DIP:DIP-14_W7.62mm_Socket
- Z34: renamed from U34; value 74LS74 -> 7474; footprint (none) -> Package_DIP:DIP-14_W7.62mm_Socket
- Z4: value 74LS20 -> 7420; footprint (none) -> Package_DIP:DIP-14_W7.62mm_Socket
- Z46, Z54: value 74LS00 -> 7400; footprint (none) -> Package_DIP:DIP-14_W7.62mm_Socket
- Z53: value 74LS02 -> 7402; footprint (none) -> Package_DIP:DIP-14_W7.62mm_Socket
- Z55: value 74LS10 -> 7410; footprint (none) -> Package_DIP:DIP-14_W7.62mm_Socket
Connections:
- net FLAG: now reaches Z15.5 (Z), Z35.13
- net ~FLAG: now reaches Z15.6 (~Z), Z35.1
- net DO_JUMP_CALL_OR_RETURN renamed FLAG_MATCH
- net JUMP_CALL_FLAG renamed JUMP_CALL_TAKE
- net ~JUMP_CALL_FLAG renamed ~JUMP_CALL_TAKE
- net ~RST_JUMP_CALL_FLAG renamed ~EXECUTE_DONE
Other:
- note added: "BRANCHING CONTROL"
- note added: "FLAG SELECT"
- note added: "PARITY FLAG"
- note added: "SIGN FLAG"
- note added: "UNCODITIONAL BRANCH"
- note added: "ZERO FLAG"
- note removed: "UNCODITIONAL JUMP/CALL/RETURN"
