File: Processor/Processor.sch (KiCad schematic (older format))
At the start: 6 parts, among them J11 Conn_02x10_Top_Bottom, J12 Conn_02x10_Top_Bottom, J13 Conn_02x10_Top_Bottom, J14 Conn_02x10_Top_Bottom, P5A Conn_02x28_Top_Bottom, P5B Conn_02x18_Top_Bottom

Commit message: Decoder 1 Rev 1
Changed lines of the file:
@@
 F10 "PHI1" O L 1400 2950 50
 F11 "PHI2" O L 1400 2850 50
-F12 "AA" I R 2700 10900 50
-F13 "W" O R 2700 2500 50
+F12 "~MEM_INDIRECT" I R 2700 10900 50
+F13 "MEM_RW" O R 2700 2500 50
 F14 "V" O R 2700 9800 50
 F15 "ENABLE_COMP" I L 1400 900 50
@@
 F22 "WORD_SELECT_SYS" O L 1400 800 50
 F23 "WORD_SELECT" O R 2700 11000 50
-F24 "~MEM.RD" I R 2700 3150 50
+F24 "~IMM_RD" I R 2700 3150 50
 F25 "IR.CLK_EN" O R 2700 3550 50
 F26 "OPCODE_HALT" I R 2700 2950 50
@@
 F9 "~RH.WR" I L 6850 7650 50
 F10 "~RL.WR" I L 6850 7750 50
-F11 "W" I L 6850 7250 50
+F11 "MEM_RW" I L 6850 7250 50
 F12 "OPCODE_REG" I R 7900 7150 50
 F13 "~OPCODE_REG" I R 7900 7250 50
@@
 F3 "RA_SER_CLK" I L 12350 3900 50
 F4 "ALU_BIT_OUT" I L 12350 4200 50
-F5 "W" I L 12350 3400 50
+F5 "MEM_RW" I L 12350 3400 50
 F6 "DC" I L 12350 4100 50
 F7 "CARRY_FLAG" I L 12350 4300 50
@@
 F16 "RA.PAR_~SER" O R 7700 3650 50
 F17 "IO.RD" O R 7700 3550 50
-F18 "W" I L 6050 3400 50
+F18 "MEM_RW" I L 6050 3400 50
 F19 "OPCODE_ALU" O R 7700 5350 50
 F20 "OPCODE_CALL_JUMP_~RETURN" O R 7700 5450 50
@@
 F3 "~DATA" O L 5500 7950 50
 F4 "PHI1_REG" I L 5500 9250 50
-F5 "W" I L 5500 8050 50
+F5 "MEM_RW" I L 5500 8050 50
 F6 "OPCODE_REG" I R 6550 8550 50
 F7 "~OPCODE_REG" I R 6550 8650 50
@@
 F15 "~OPCODE00n" O R 4950 3800 50
 F16 "~ALU_SHIFT" O R 4950 4250 50
-F17 "~MEM.RD" O R 4950 6750 50
+F17 "~IMM_RD" O R 4950 6750 50
 F18 "~RH.RD" O R 4950 7400 50
 F19 "~RA.RD" O R 4950 6500 50
-F20 "~MEM.WR" O R 4950 6850 50
+F20 "~IMM_WR" O R 4950 6850 50
 F21 "~RL.WR" O R 4950 7750 50
 F22 "~RH.WR" O R 4950 7650 50
@@
 F0 "ALU" 50
 F1 "ALU.sch" 50
-F2 "W" I L 9550 3500 50
+F2 "MEM_RW" I L 9550 3500 50
 F3 "DC" O R 10950 4100 50
 F4 "AW" I L 9550 3600 50
@@
 Text Notes -3150 8400 0    50   ~ 0
 J
-Text GLabel -1500 4550 0    50   Output ~ 0
+Text GLabel -1500 4550 0    50   Input ~ 0
 ~POR_OUT
 Text GLabel -800 4450 2    50   Input ~ 0
@@
 Text GLabel -1500 4650 0    50   Output ~ 0
 STROBE_1
-Text GLabel -3350 5550 0    50   Output ~ 0
+Text GLabel -3350 5550 0    50   Input ~ 0
 I4
-Text GLabel -3350 4850 0    50   Output ~ 0
+Text GLabel -3350 4850 0    50   Input ~ 0
 I3
 Text GLabel -1500 3550 0    50   Output ~ 0
 I2
-Text GLabel -1500 3850 0    50   Output ~ 0
+Text GLabel -1500 3850 0    50   Input ~ 0
 I1
 Text Notes -2750 3850 0    50   ~ 0
@@
 Text GLabel -3350 3950 0    50   Output ~ 0
 A7_IN
-Text GLabel -3350 4950 0    50   Output ~ 0
+Text GLabel -3350 4950 0    50   Input ~ 0
 IO_READ
-Text GLabel -2650 4550 2    50   Output ~ 0
+Text GLabel -2650 4550 2    50   Input ~ 0
 A0_OUT
-Text GLabel -3350 4350 0    50   Output ~ 0
+Text GLabel -3350 4350 0    50   Input ~ 0
 A1_OUT
-Text GLabel -2650 4350 2    50   Output ~ 0
+Text GLabel -2650 4350 2    50   Input ~ 0
 A2_OUT
-Text GLabel -2650 4450 2    50   Output ~ 0
+Text GLabel -2650 4450 2    50   Input ~ 0
 A3_OUT
-Text GLabel -2650 3750 2    50   Output ~ 0
+Text GLabel -2650 3750 2    50   Input ~ 0
 A4_OUT
-Text GLabel -2650 3850 2    50   Output ~ 0
+Text GLabel -2650 3850 2    50   Input ~ 0
 A5_OUT
-Text GLabel -2650 3950 2    50   Output ~ 0
+Text GLabel -2650 3950 2    50   Input ~ 0
 A6_OUT
-Text GLabel -3350 4450 0    50   Output ~ 0
+Text GLabel -3350 4450 0    50   Input ~ 0
 A7_OUT
-Text GLabel -3350 4750 0    50   Output ~ 0
+Text GLabel -3350 4750 0    50   Input ~ 0
 CB0
-Text GLabel -3350 4650 0    50   Output ~ 0
+Text GLabel -3350 4650 0    50   Input ~ 0
 CB1
-Text GLabel -2650 3650 2    50   Output ~ 0
+Text GLabel -2650 3650 2    50   Input ~ 0
 CB2
-Text GLabel -2650 4750 2    50   Output ~ 0
+Text GLabel -2650 4750 2    50   Input ~ 0
 CB3
-Text GLabel -2650 4250 2    50   Output ~ 0
+Text GLabel -2650 4250 2    50   Input ~ 0
 CB4
-Text GLabel -2650 4150 2    50   Output ~ 0
+Text GLabel -2650 4150 2    50   Input ~ 0
 CB5
-Text GLabel -2650 4050 2    50   Output ~ 0
+Text GLabel -2650 4050 2    50   Input ~ 0
 CB6
-Text GLabel -2650 4650 2    50   Output ~ 0
+Text GLabel -2650 4650 2    50   Input ~ 0
 CB7
 Text Notes -2750 3650 0    50   ~ 0
@@
 Text Notes -2650 5850 0    50   ~ 0
 SPARE
-Text GLabel -2650 5950 2    50   Output ~ 0
+Text GLabel -2650 5950 2    50   Input ~ 0
 ~ENABLE_1
-Text GLabel -2650 6050 2    50   Output ~ 0
+Text GLabel -2650 6050 2    50   Input ~ 0
 ~ENABLE_2
 Text Notes -2750 4950 0    50   ~ 0
@@
 F3 "PHASE_CLOCK" I L 14600 9300 50
 F4 "CW" I L 14600 5850 50
-F5 "AA" O L 14600 10900 50
+F5 "~MEM_INDIRECT" O L 14600 10900 50
 F6 "ST.DIR" O L 14600 8450 50
 F7 "ST.COUNT" O L 14600 8350 50
@@
 F12 "STROBE_2" I L 14600 8750 50
 F13 "WORD_SELECT" I L 14600 11000 50
-F14 "~MEM.RD" I L 14600 6750 50
+F14 "~IMM_RD" I L 14600 6750 50
 F15 "A" O L 14600 11100 50
-F16 "~MEM.WR" I L 14600 6850 50
+F16 "~IMM_WR" I L 14600 6850 50
 F17 "STROBE_4" I L 14600 8850 50
-F18 "W" I L 14600 2950 50
+F18 "MEM_RW" I L 14600 2950 50
 F19 "STROBE_1" I L 14600 8650 50
 F20 "AW" I L 14600 3050 50
@@
 Wire Wire Line
 	14050 4850 14050 10300
+Text Notes -3150 8100 0    50   ~ 0
+E
 $EndSCHEMATC

Commit message: Schematics for display & keyboard, adding LEDs to processor PCB
Parts:
- removed P5A: Conn_02x28_Top_Bottom, symbol Connector_Generic:Conn_02x28_Top_Bottom
- removed P5B: Conn_02x18_Top_Bottom, symbol Connector_Generic:Conn_02x18_Top_Bottom
- added PAB5: Edge P5A Bottom, Datapoint2200:EdgeConn_28_Pin_Pitch_3.96mm, symbol Connector:Conn_01x28_Male
- added PAT5: Edge P5A Top, Datapoint2200:EdgeConn_28_Pin_Pitch_3.96mm, symbol Connector:Conn_01x28_Male
- added PBB5: Edge P5B Bottom, Datapoint2200:EdgeConn_18_Pin_Pitch_3.96mm, symbol Connector:Conn_01x18_Male
- added PBT5: Edge P5B Top, Datapoint2200:EdgeConn_18_Pin_Pitch_3.96mm, symbol Connector:Conn_01x18_Male
- J11, J12, J13, J14: footprint (none) -> Datapoint2200:EdgeConn_Socket_20_Pin_Pitch_3.96mm
Connections:
- net +12V: now also J11.14 (Pin_14), J12.14 (Pin_14), J13.14 (Pin_14), J14.14 (Pin_14), PAB5.23 (Pin_23), PAT5.23 (Pin_23)
- net +5V: now also J11.15 (Pin_15), J11.5 (Pin_5), J12.15 (Pin_15), J12.5 (Pin_5), J13.15 (Pin_15), J13.5 (Pin_5), J14.15 (Pin_15), J14.5 (Pin_5), PAB5.2 (Pin_2), PAT5.2 (Pin_2), PBB5.17 (Pin_17), PBT5.17 (Pin_17)
- net -12V: now also J11.19 (Pin_19), J11.9 (Pin_9), J12.19 (Pin_19), J12.9 (Pin_9), J13.19 (Pin_19), J13.9 (Pin_9), J14.19 (Pin_19), J14.9 (Pin_9), PAB5.28 (Pin_28), PAT5.28 (Pin_28)
- net -5V: now also J11.10 (Pin_10), J11.20 (Pin_20), J12.10 (Pin_10), J12.20 (Pin_20), J13.10 (Pin_10), J13.20 (Pin_20), J14.10 (Pin_10), J14.20 (Pin_20), PBB5.1 (Pin_1), PBT5.1 (Pin_1)
- net CB0: now also PAT5.14 (Pin_14)
- net CB1: now also PAT5.13 (Pin_13)
- net CB2: now also PAB5.3 (Pin_3)
- net CB3: now also PAB5.14 (Pin_14)
- net CB4: now also PAB5.9 (Pin_9)
- net CB5: now also PAB5.8 (Pin_8)
- net CB6: now also PAB5.7 (Pin_7)
- net CB7: now also PAB5.13 (Pin_13)
- net DIV64_CLK: now also PBT5.8 (Pin_8)
- net ENABLE_COMP: now also PBT5.10 (Pin_10)
- net EOR_REBOOT: now also PBT5.7 (Pin_7)
- net GND: now also J11.4 (Pin_4), J12.4 (Pin_4), J13.4 (Pin_4), J14.4 (Pin_4), PAB5.1 (Pin_1), PAT5.1 (Pin_1), PBB5.18 (Pin_18), PBT5.18 (Pin_18)
- net I1: now also PBT5.5 (Pin_5)
- net I2: now also PBT5.2 (Pin_2)
- net I3: now also PAT5.15 (Pin_15)
- net I4: now also PAT5.22 (Pin_22)
- net INC_P: now also PBT5.6 (Pin_6)
- net INH_MEMORY: now also PBT5.3 (Pin_3)
- net IO_READ: now also PAT5.16 (Pin_16)
- net MEM_INPUTS: now also J11.16 (Pin_16), J12.16 (Pin_16), J13.16 (Pin_16), J14.16 (Pin_16)
- net MEM_READ: now also J11.18 (Pin_18), J12.18 (Pin_18), J13.18 (Pin_18), J14.18 (Pin_18)
- net MEM_WRITE: now also J11.17 (Pin_17), J12.17 (Pin_17), J13.17 (Pin_17), J14.17 (Pin_17)
- net P10: now also J11.12 (Pin_12), J12.12 (Pin_12), J13.12 (Pin_12), J14.12 (Pin_12)
- net P11: now also PBB5.3 (Pin_3)
- net P12: now also PBB5.2 (Pin_2)
- net P6: now also J11.3 (Pin_3), J12.3 (Pin_3), J13.3 (Pin_3), J14.3 (Pin_3)
- net P7: now also J11.2 (Pin_2), J12.2 (Pin_2), J13.2 (Pin_2), J14.2 (Pin_2)
- net P8: now also J11.1 (Pin_1), J12.1 (Pin_1), J13.1 (Pin_1), J14.1 (Pin_1)
- net P9: now also J11.13 (Pin_13), J12.13 (Pin_13), J13.13 (Pin_13), J14.13 (Pin_13)
- net PHASE_CLOCK: now also PBB5.16 (Pin_16)
- net PHI1: now also J11.8 (Pin_8), J12.8 (Pin_8), J13.8 (Pin_8), J14.8 (Pin_8)
- net PHI1_MEM: now also PAT5.20 (Pin_20)
- net PHI1_REG: now also PAT5.24 (Pin_24)
- net PHI2: now also J11.6 (Pin_6), J12.6 (Pin_6), J13.6 (Pin_6), J14.6 (Pin_6)
- net PHI2_MEM: now also PAT5.21 (Pin_21)
- net RUN_SW: now also PBT5.9 (Pin_9)
- net STROBE_1: now also PBT5.13 (Pin_13)
- net STROBE_2: now also PAT5.19 (Pin_19)
- net STROBE_3: now also PBT5.11 (Pin_11)
- net STROBE_4: now also PAT5.17 (Pin_17)
- net ~ENABLE_1: now also PAB5.26 (Pin_26)
- net ~ENABLE_2: now also PAB5.27 (Pin_27)
- net ~EOR_REBOOT: now also PBT5.14 (Pin_14)
- net ~HALT_LIGHT: now also PBB5.14 (Pin_14)
- net ~MEM_WRITE_READY: now also PAT5.25 (Pin_25)
- net ~POR_IN: now also PBT5.16 (Pin_16)
- net ~POR_OUT: now also PBT5.12 (Pin_12)
- net ~RESET_P: now also PBT5.15 (Pin_15)
- net ~RUN_LIGHT: now also PBB5.13 (Pin_13)
- net ~PAGE_SELECT_1: now reaches J11.11 (Pin_11)
- net ~MEM_OUTPUTS: now reaches J11.7 (Pin_7)
- net ~MEM_OUTPUTS: now also J12.7 (Pin_7), J13.7 (Pin_7), J14.7 (Pin_7)
- net ~PAGE_SELECT_2: now reaches J12.11 (Pin_11)
- net ~PAGE_SELECT_3: now reaches J13.11 (Pin_11)
- net ~PAGE_SELECT_4: now reaches J14.11 (Pin_11)
- new net AIN0: PAT5.12 (Pin_12)
- new net AIN1: PAT5.9 (Pin_9)
- new net AIN2: PAT5.8 (Pin_8)
- new net AIN3: PAT5.7 (Pin_7)
- new net AIN4: PAT5.5 (Pin_5)
- new net AIN5: PAT5.3 (Pin_3)
- new net AIN6: PAT5.4 (Pin_4)
- new net AIN7: PAT5.6 (Pin_6)
- new net AOUT0: PAB5.12 (Pin_12)
- new net AOUT1: PAT5.10 (Pin_10)
- new net AOUT2: PAB5.10 (Pin_10)
- new net AOUT3: PAB5.11 (Pin_11)
- new net AOUT4: PAB5.4 (Pin_4)
- new net AOUT5: PAB5.5 (Pin_5)
- new net AOUT6: PAB5.6 (Pin_6)
- new net AOUT7: PAT5.11 (Pin_11)
- new net WORD_SELECT_SYS: PBB5.11 (Pin_11)
- new net ~HALT: PBB5.15 (Pin_15)
- new net ~REBOOT_SERIAL_DATA: PAT5.18 (Pin_18)
- no-connect marks 0 -> 21
Other:
- note removed: "G"
- moved on the sheet: J11
