File: Processor/Registers1.sch (KiCad schematic (older format))
At the start: 10 parts

Commit message: Decoder 1 Rev 1
Connections:
- net W renamed MEM_RW
Changed lines of the file:
@@
 Wire Wire Line
 	7400 1700 7800 1700
-Text HLabel 3350 3200 0    50   Input ~ 0
-W
+Text HLabel 3250 3200 0    50   Input ~ 0
+MEM_RW
 Wire Wire Line
-	3450 3200 3350 3200
+	3450 3200 3250 3200
 Wire Wire Line
 	7300 3100 7300 1600

Commit message: Schematics for display & keyboard, adding LEDs to processor PCB
Parts:
- R25, R31, R56: footprint (none) -> Resistor_THT:R_Axial_DIN0207_L6.3mm_D2.5mm_P10.16mm_Horizontal
- Z3: value 74LS20 -> 7420; footprint (none) -> Package_DIP:DIP-14_W7.62mm_Socket
- Z41: value 74LS02 -> 7402; footprint (none) -> Package_DIP:DIP-14_W7.62mm_Socket
- Z59: value 74LS06 -> 7406; footprint (none) -> Package_DIP:DIP-14_W7.62mm_Socket; symbol 74xx:74LS06 -> Datapoint2200:74LS06
- Z60: value 74LS03 -> 7403; footprint (none) -> Package_DIP:DIP-14_W7.62mm_Socket; symbol 74xx:74LS03 -> Datapoint2200:74LS03
- Z61: value 74LS00 -> 7400; footprint (none) -> Package_DIP:DIP-14_W7.62mm_Socket
- Z62, Z66: value 74HC164 -> 74164; footprint (none) -> Package_DIP:DIP-14_W7.62mm_Socket
Connections:
- net RH7: now reaches Z62.3 (Q0)
- net RH6: now reaches Z62.4 (Q1)
- net RH5: now reaches Z62.5 (Q2)
- net D_REG_IN renamed REG_DATA
- no-connect marks 3 -> 0
Other:
- note added: "RH5 to RH7 only\nrequired for LEDs"
- note added: "~DATA~ is the main data bus in the system. Data\ncan be written to this line by any of the registers,\nthe memory cards (~MEM_OUTPUTS~) or by the\ntape cards (~REBOOT_SERIAL_DATA~).\n\n~DATA~ is inverted here to:\nREG_DATA as inputs to the registers.\nDATA: as general data in the processor.\n\nIt is also inverted and send to the memory\ncards (~MEM_INPUTS~)."
Changed lines of the file:
@@
 $Descr A4 11693 8268
 encoding utf-8
-Sheet 4 12
+Sheet 4 21
 Title ""
 Date ""
@@
 $EndDescr
 $Comp
-L 74xx:74LS06 Z59
+L Datapoint2200:74LS06 Z59
 U 6 1 62453E75
 P 1850 1400
 F 0 "Z59" H 1850 1717 50  0000 C CNN
-F 1 "74LS06" H 1850 1626 50  0000 C CNN
-F 2 "" H 1850 1400 50  0001 C CNN
+F 1 "7406" H 1850 1626 50  0000 C CNN
+F 2 "Package_DIP:DIP-14_W7.62mm_Socket" H 1850 1400 50  0001 C CNN
 F 3 "http://www.ti.com/lit/gpn/sn74LS06" H 1850 1400 50  0001 C CNN
 	6    1850 1400
@@
 $EndComp
 $Comp
-L 74xx:74LS06 Z59
+L Datapoint2200:74LS06 Z59
 U 1 1 6245427C
 P 1850 1900
 F 0 "Z59" H 1850 2217 50  0000 C CNN
-F 1 "74LS06" H 1850 2126 50  0000 C CNN
-F 2 "" H 1850 1900 50  0001 C CNN
+F 1 "7406" H 1850 2126 50  0000 C CNN
+F 2 "Package_DIP:DIP-14_W7.62mm_Socket" H 1850 1900 50  0001 C CNN
 F 3 "http://www.ti.com/lit/gpn/sn74LS06" H 1850 1900 50  0001 C CNN
 	1    1850 1900
@@
 F 0 "R25" V 1850 2100 50  0000 L CNN
 F 1 "1k" V 1750 2100 50  0000 L CNN
-F 2 "" V 1680 2200 50  0001 C CNN
+F 2 "Resistor_THT:R_Axial_DIN0207_L6.3mm_D2.5mm_P10.16mm_Horizontal" V 1680 2200 50  0001 C CNN
 F 3 "~" H 1750 2200 50  0001 C CNN
 	1    1750 2200
@@
 Connection ~ 1450 1900
 $Comp
-L power:+5V #PWR?
+L power:+5V #PWR0215
 U 1 1 624554E4
 P 2000 2200
-F 0 "#PWR?" H 2000 2050 50  0001 C CNN
+F 0 "#PWR0215" H 2000 2050 50  0001 C CNN
 F 1 "+5V" H 2100 2250 50  0000 C CNN
 F 2 "" H 2000 2200 50  0001 C CNN
@@
 F 0 "R56" V 2600 1900 50  0000 L CNN
 F 1 "470" V 2500 1900 50  0000 L CNN
-F 2 "" V 2430 2000 50  0001 C CNN
+F 2 "Resistor_THT:R_Axial_DIN0207_L6.3mm_D2.5mm_P10.16mm_Horizontal" V 2430 2000 50  0001 C CNN
 F 3 "~" H 2500 2000 50  0001 C CNN
 	1    2500 2000
@@
 F 0 "R31" V 2600 1400 50  0000 L CNN
 F 1 "470" V 2500 1400 50  0000 L CNN
-F 2 "" V 2430 1500 50  0001 C CNN
+F 2 "Resistor_THT:R_Axial_DIN0207_L6.3mm_D2.5mm_P10.16mm_Horizontal" V 2430 1500 50  0001 C CNN
 F 3 "~" H 2500 1500 50  0001 C CNN
 	1    2500 1500
@@
 $EndComp
 $Comp
-L power:+5V #PWR?
+L power:+5V #PWR0216
 U 1 1 624566F7
 P 2750 2000
-F 0 "#PWR?" H 2750 1850 50  0001 C CNN
+F 0 "#PWR0216" H 2750 1850 50  0001 C CNN
 F 1 "+5V" H 2850 2050 50  0000 C CNN
 F 2 "" H 2750 2000 50  0001 C CNN
@@
 $EndComp
 $Comp
-L power:+5V #PWR?
+L power:+5V #PWR0217
 U 1 1 624569F8
 P 2750 1500
-F 0 "#PWR?" H 2750 1350 50  0001 C CNN
+F 0 "#PWR0217" H 2750 1350 50  0001 C CNN
 F 1 "+5V" H 2850 1550 50  0000 C CNN
 F 2 "" H 2750 1500 50  0001 C CNN
@@
 P 4200 1650
 F 0 "Z3" H 4200 1308 50  0000 C CNN
-F 1 "74LS20" H 4200 1399 50  0000 C CNN
-F 2 "" H 4200 1650 50  0001 C CNN
+F 1 "7420" H 4200 1399 50  0000 C CNN
+F 2 "Package_DIP:DIP-14_W7.62mm_Socket" H 4200 1650 50  0001 C CNN
 F 3 "http://www.ti.com/lit/gpn/sn74LS20" H 4200 1650 50  0001 C CNN
 	2    4200 1650
@@
 P 4200 2400
 F 0 "Z61" H 4200 2725 50  0000 C CNN
-F 1 "74LS00" H 4200 2634 50  0000 C CNN
-F 2 "" H 4200 2400 50  0001 C CNN
+F 1 "7400" H 4200 2634 50  0000 C CNN
+F 2 "Package_DIP:DIP-14_W7.62mm_Socket" H 4200 2400 50  0001 C CNN
 F 3 "http://www.ti.com/lit/gpn/sn74ls00" H 4200 2400 50  0001 C CNN
 	4    4200 2400
@@
 P 4200 3400
 F 0 "Z41" H 4200 3083 50  0000 C CNN
-F 1 "74LS02" H 4200 3174 50  0000 C CNN
-F 2 "" H 4200 3400 50  0001 C CNN
+F 1 "7402" H 4200 3174 50  0000 C CNN
+F 2 "Package_DIP:DIP-14_W7.62mm_Socket" H 4200 3400 50  0001 C CNN
 F 3 "http://www.ti.com/lit/gpn/sn74ls02" H 4200 3400 50  0001 C CNN
 	4    4200 3400
@@
 P 5450 2400
 F 0 "Z66" V 5550 2850 50  0000 L CNN
-F 1 "74HC164" V 5650 2850 50  0000 L CNN
-F 2 "" H 6350 2100 50  0001 C CNN
+F 1 "74164" V 5650 2850 50  0000 L CNN
+F 2 "Package_DIP:DIP-14_W7.62mm_Socket" H 6350 2100 50  0001 C CNN
 F 3 "https://assets.nexperia.com/documents/data-sheet/74HC_HCT164.pdf" H 6350 2100 50  0001 C CNN
 	1    5450 2400
@@
 $EndComp
 $Comp
-L power:+5V #PWR?
+L power:+5V #PWR0218
 U 1 1 6245E8DA
 P 5950 2400
-F 0 "#PWR?" H 5950 2250 50  0001 C CNN
+F 0 "#PWR0218" H 5950 2250 50  0001 C CNN
 F 1 "+5V" H 6050 2450 50  0000 C CNN
 F 2 "" H 5950 2400 50  0001 C CNN
@@
 $EndComp
 $Comp
-L power:GND #PWR?
+L power:GND #PWR0219
 U 1 1 6245EDB9
 P 4850 2400
-F 0 "#PWR?" H 4850 2150 50  0001 C CNN
+F 0 "#PWR0219" H 4850 2150 50  0001 C CNN
 F 1 "GND" H 4855 2227 50  0001 C CNN
 F 2 "" H 4850 2400 50  0001 C CNN
@@
 	5150 1650 5150 2000
 $Comp
-L power:+5V #PWR?
+L power:+5V #PWR0220
 U 1 1 62462FAD
 P 5650 2000
-F 0 "#PWR?" H 5650 1850 50  0001 C CNN
+F 0 "#PWR0220" H 5650 1850 50  0001 C CNN
 F 1 "+5V" H 5750 2050 50  0001 C CNN
 F 2 "" H 5650 2000 50  0001 C CNN
@@
 $EndComp
 $Comp
-L 74xx:74LS03 Z60
+L Datapoint2200:74LS03 Z60
 U 3 1 624632F0
 P 6800 2400
 F 0 "Z60" H 6800 2725 50  0000 C CNN
-F 1 "74LS03" H 6800 2634 50  0000 C CNN
-F 2 "" H 6800 2400 50  0001 C CNN
+F 1 "7403" H 6800 2634 50  0000 C CNN
+F 2 "Package_DIP:DIP-14_W7.62mm_Socket" H 6800 2400 50  0001 C CNN
 F 3 "http://www.ti.com/lit/gpn/sn74LS03" H 6800 2400 50  0001 C CNN
 	3    6800 2400
@@
 P 8100 1650
 F 0 "Z3" H 8100 2025 50  0000 C CNN
-F 1 "74LS20" H 8100 1934 50  0000 C CNN
-F 2 "" H 8100 1650 50  0001 C CNN
+F 1 "7420" H 8100 1934 50  0000 C CNN
+F 2 "Package_DIP:DIP-14_W7.62mm_Socket" H 8100 1650 50  0001 C CNN
 F 3 "http://www.ti.com/lit/gpn/sn74LS20" H 8100 1650 50  0001 C CNN
 	1    8100 1650
@@
 P 8100 2350
 F 0 "Z61" H 8100 2675 50  0000 C CNN
-F 1 "74LS00" H 8100 2584 50  0000 C CNN
-F 2 "" H 8100 2350 50  0001 C CNN
+F 1 "7400" H 8100 2584 50  0000 C CNN
+F 2 "Package_DIP:DIP-14_W7.62mm_Socket" H 8100 2350 50  0001 C CNN
 F 3 "http://www.ti.com/lit/gpn/sn74ls00" H 8100 2350 50  0001 C CNN
 	3    8100 2350
@@
 P 8100 3400
 F 0 "Z41" H 8100 3725 50  0000 C CNN
-F 1 "74LS02" H 8100 3634 50  0000 C CNN
-F 2 "" H 8100 3400 50  0001 C CNN
+F 1 "7402" H 8100 3634 50  0000 C CNN
+F 2 "Package_DIP:DIP-14_W7.62mm_Socket" H 8100 3400 50  0001 C CNN
 F 3 "http://www.ti.com/lit/gpn/sn74ls02" H 8100 3400 50  0001 C CNN
 	3    8100 3400
@@
 P 9200 2400
 F 0 "Z62" V 9300 2850 50  0000 L CNN
-F 1 "74HC164" V 9400 2850 50  0000 L CNN
-F 2 "" H 10100 2100 50  0001 C CNN
+F 1 "74164" V 9400 2850 50  0000 L CNN
+F 2 "Package_DIP:DIP-14_W7.62mm_Socket" H 10100 2100 50  0001 C CNN
 F 3 "https://assets.nexperia.com/documents/data-sheet/74HC_HCT164.pdf" H 10100 2100 50  0001 C CNN
 	1    9200 2400
@@
 $EndComp
 $Comp
-L power:GND #PWR?
+L power:GND #PWR0221
 U 1 1 6249FCE8
 P 8600 2400
-F 0 "#PWR?" H 8600 2150 50  0001 C CNN
+F 0 "#PWR0221" H 8600 2150 50  0001 C CNN
 F 1 "GND" H 8605 2227 50  0001 C CNN
 F 2 "" H 8600 2400 50  0001 C CNN
@@
 $EndComp
 $Comp
-L power:+5V #PWR?
+L power:+5V #PWR0222
 U 1 1 624A026D
 P 9700 2400
-F 0 "#PWR?" H 9700 2250 50  0001 C CNN
+F 0 "#PWR0222" H 9700 2250 50  0001 C CNN
 F 1 "+5V" H 9800 2450 50  0000 C CNN
 F 2 "" H 9700 2400 50  0001 C CNN
@@
 Connection ~ 9100 1900
 Text HLabel 3150 1400 1    50   Output ~ 0
-D_REG_IN
+REG_DATA
 Wire Wire Line
 	8400 1650 8900 1650
@@
 	8900 1650 8900 2000
 $Comp
-L power:+5V #PWR?
+L power:+5V #PWR0223
 U 1 1 624AF4BE
 P 9400 2000
-F 0 "#PWR?" H 9400 1850 50  0001 C CNN
+F 0 "#PWR0223" H 9400 1850 50  0001 C CNN
 F 1 "+5V" H 9500 2050 50  0001 C CNN
 F 2 "" H 9400 2000 50  0001 C CNN
@@
 	1    0    0    -1
 $EndComp
-NoConn ~ 9500 2800
-NoConn ~ 9400 2800
-NoConn ~ 9300 2800
-$Comp
-L 74xx:74LS03 Z60
+$Comp
+L Datapoint2200:74LS03 Z60
 U 4 1 624B6B83
 P 10500 2400
 F 0 "Z60" H 10500 2725 50  0000 C CNN
-F 1 "74LS03" H 10500 2634 50  0000 C CNN
-F 2 "" H 10500 2400 50  0001 C CNN
+F 1 "7403" H 10500 2634 50  0000 C CNN
+F 2 "Package_DIP:DIP-14_W7.62mm_Socket" H 10500 2400 50  0001 C CNN
 F 3 "http://www.ti.com/lit/gpn/sn74LS03" H 10500 2400 50  0001 C CNN
 	4    10500 2400
@@
 	8800 3750 8800 2900
 Connection ~ 8800 2900
-Text GLabel 5850 3850 3    50   Input ~ 0
+Text GLabel 5950 3850 2    50   Output ~ 0
 RL[0..7]
-Text GLabel 9300 3850 3    50   Input ~ 0
-RH[0..4]
-Text HLabel 5950 3850 2    50   Output ~ 0
-RL_BUS
-Text HLabel 9450 3850 2    50   Output ~ 0
+Text GLabel 9550 3850 3    50   Output ~ 0
+RH[0..7]
+Text HLabel 9650 3850 2    50   Output ~ 0
 RH_BUS
 Wire Wire Line
@@
 	3250 3600 3800 3600
 Connection ~ 3800 3600
+Text Notes 1100 4750 0    50   ~ 0
+~DATA~ is the main data bus in the system. Data\ncan be written to this line by any of the registers,\nthe memory cards (~MEM_OUTPUTS~) or by the\ntape cards (~REBOOT_SERIAL_DATA~).\n\n~DATA~ is inverted here to:\nREG_DATA as inputs to the registers.\nDATA: as general data in the processor.\n\nIt is also inverted and send to the memory\ncards (~MEM_INPUTS~).
+$Sheet
+S 7650 5150 750  550
+U 64EF8E46
+F0 "Reg1Blinken" 50
+F1 "Reg1Blinken.sch" 50
+F2 "RHBUS" I L 7650 5250 50
+F3 "RLBUS" I L 7650 5350 50
+$EndSheet
+Text GLabel 7550 5350 0    50   Input ~ 0
+RL[0..7]
+Text GLabel 7550 5250 0    50   Input ~ 0
+RH[0..7]
+Wire Wire Line
+	7550 5250 7650 5250
+Wire Wire Line
+	7550 5350 7650 5350
+Entry Wire Line
+	9300 3750 9200 3850
+Entry Wire Line
+	9400 3750 9300 3850
+Entry Wire Line
+	9500 3750 9400 3850
+Wire Wire Line
+	9300 2800 9300 3750
+Wire Wire Line
+	9400 2800 9400 3750
+Wire Wire Line
+	9500 2800 9500 3750
+Text Label 9300 3750 1    50   ~ 0
+RH5
+Text Label 9400 3750 1    50   ~ 0
+RH6
+Text Label 9500 3750 1    50   ~ 0
+RH7
+Text Notes 9650 3700 0    50   ~ 0
+RH5 to RH7 only\nrequired for LEDs
 Wire Bus Line
-	8700 3850 9450 3850
+	8700 3850 9650 3850
 Wire Bus Line
 	4950 3850 5950 3850
