File: Processor/Registers2.sch (KiCad schematic (older format))
At the start: 9 parts

Commit message: Decoder 1 Rev 1
Connections:
- net W renamed MEM_RW
Changed lines of the file:
@@
 	950  1500 1500 1500
 Text HLabel 850  2950 0    50   Input ~ 0
-W
+MEM_RW
 Wire Wire Line
 	1500 1600 1050 1600

Commit message: Schematics for display & keyboard, adding LEDs to processor PCB
Parts:
- Z19, Z38: value 74LS20 -> 7420; footprint (none) -> Package_DIP:DIP-14_W7.62mm_Socket
- Z20, Z21, Z39, Z40: value 74HC164 -> 74164; footprint (none) -> Package_DIP:DIP-14_W7.62mm_Socket
- Z22: value 74LS00 -> 7403; footprint (none) -> Package_DIP:DIP-14_W7.62mm_Socket; symbol 74xx:74LS03 -> Datapoint2200:74LS03
- Z22: value 74LS00 -> 7403; footprint (none) -> Package_DIP:DIP-14_W7.62mm_Socket; symbol 74xx:74LS00 -> Datapoint2200:74LS03
- Z23: value 74LS02 -> 7402; footprint (none) -> Package_DIP:DIP-14_W7.62mm_Socket
- Z42: value 74LS00 -> 7400; footprint (none) -> Package_DIP:DIP-14_W7.62mm_Socket
Connections:
- net MEM_RW: now also Z38.4; no longer Z38.5
- net OPCODE_REG: now also Z38.5; no longer Z38.4
- net RD3: now reaches Z20.10 (Q4)
- net RD2: now reaches Z20.11 (Q5)
- net RD1: now reaches Z20.12 (Q6)
- net RD0: now reaches Z20.13 (Q7), Z22.2
- net RD7: now reaches Z20.3 (Q0)
- net RD6: now reaches Z20.4 (Q1)
- net RD5: now reaches Z20.5 (Q2)
- net RD4: now reaches Z20.6 (Q3)
- net RE3: now reaches Z21.10 (Q4)
- net RE2: now reaches Z21.11 (Q5)
- net RE1: now reaches Z21.12 (Q6)
- net RE0: now reaches Z21.13 (Q7), Z22.12
- net RE7: now reaches Z21.3 (Q0)
- net RE6: now reaches Z21.4 (Q1)
- net RE5: now reaches Z21.5 (Q2)
- net RE4: now reaches Z21.6 (Q3)
- net RB3: now reaches Z40.10 (Q4)
- net RB2: now reaches Z40.11 (Q5)
- net RB1: now reaches Z40.12 (Q6)
- net RB0: now reaches Z22.9, Z40.13 (Q7)
- net RB7: now reaches Z40.3 (Q0)
- net RB6: now reaches Z40.4 (Q1)
- net RB5: now reaches Z40.5 (Q2)
- net RB4: now reaches Z40.6 (Q3)
- net RC3: now reaches Z39.10 (Q4)
- net RC2: now reaches Z39.11 (Q5)
- net RC1: now reaches Z39.12 (Q6)
- net RC0: now reaches Z22.4, Z39.13 (Q7)
- net RC7: now reaches Z39.3 (Q0)
- net RC6: now reaches Z39.4 (Q1)
- net RC5: now reaches Z39.5 (Q2)
- net RC4: now reaches Z39.6 (Q3)
- net D_REG_IN renamed REG_DATA
- no-connect marks 28 -> 0
Other:
- moved on the sheet: Z23A, Z23B, Z23C, Z23D
