File: Processor/Timing.sch (KiCad schematic (older format))
At the start: 43 parts, among them U48 74LS05, U59 74LS06

Commit message: Decoder 1 Rev 1
Connections:
- net AA renamed ~MEM_INDIRECT
- net W renamed MEM_RW
- net ~MEM.RD renamed ~IMM_RD
Changed lines of the file:
@@
 Wire Wire Line
 	3150 2750 2700 2750
-Text HLabel 2950 2950 0    50   Input ~ 0
-AA
-Wire Wire Line
-	2950 2950 3150 2950
+Text HLabel 3050 2950 3    50   Input ~ 0
+~MEM_INDIRECT
+Wire Wire Line
+	3050 2950 3150 2950
 Text HLabel 3850 2750 1    50   Output ~ 0
-W
+MEM_RW
 Wire Wire Line
 	3850 2850 3750 2850
@@
 $EndComp
 Text HLabel 9700 1950 0    50   Input ~ 0
-~MEM.RD
+~IMM_RD
 Wire Wire Line
 	9050 4850 9550 4850
@@
 OPCODE_ENABLE
 Text GLabel 4000 7450 0    50   Input ~ 0
-W
+MEM_RW
 Text Notes 13600 2950 0    100  ~ 0
 Run/Halt

Commit message: Schematics for display & keyboard, adding LEDs to processor PCB
Parts:
- removed C54: 100u, symbol Device:CP
- added C54: 100p 1kV, Capacitor_THT:C_Disc_D7.0mm_W2.5mm_P5.00mm, symbol Device:C
- added J901: ~WORD_SELECT, Connector_PinHeader_2.54mm:PinHeader_1x01_P2.54mm_Horizontal, symbol Connector:Conn_01x01_Male
- C56: value .001 -> .001 1kV; footprint (none) -> Capacitor_THT:C_Disc_D7.0mm_W2.5mm_P5.00mm
- C57: value 470p -> 470p 1kV; footprint (none) -> Capacitor_THT:C_Disc_D7.0mm_W2.5mm_P5.00mm
- R52, R53, R57, R58, R59, R60, R64, R66: footprint (none) -> Resistor_THT:R_Axial_DIN0207_L6.3mm_D2.5mm_P10.16mm_Horizontal
- R63: value 470 -> 220; footprint (none) -> Resistor_THT:R_Axial_DIN0207_L6.3mm_D2.5mm_P10.16mm_Horizontal
- TP1: footprint (none) -> TestPoint:TestPoint_THTPad_1.5x1.5mm_Drill0.7mm
- Z101: value 74LS193 -> 74193; footprint (none) -> Package_DIP:DIP-16_W7.62mm_Socket
- Z102: renamed from Z104; value 74LS04 -> 7404; footprint (none) -> Package_DIP:DIP-14_W7.62mm_Socket
- Z102, Z30, Z49, Z7: value 74LS04 -> 7404; footprint (none) -> Package_DIP:DIP-14_W7.62mm_Socket
- Z103, Z29: value 74LS03 -> 7403; footprint (none) -> Package_DIP:DIP-14_W7.62mm_Socket; symbol 74xx:74LS03 -> Datapoint2200:74LS03
- Z108, Z14: value 74LS40 -> 7440; footprint (none) -> Package_DIP:DIP-14_W7.62mm_Socket
- Z114, Z115: value 74LS85 -> 7485; footprint (none) -> Package_DIP:DIP-16_W7.62mm_Socket
- Z116: value 74LS08 -> 7408; footprint (none) -> Package_DIP:DIP-14_W7.62mm_Socket
- Z12, Z68, Z86: value 74LS00 -> 7400; footprint (none) -> Package_DIP:DIP-14_W7.62mm_Socket
- Z31, Z32, Z52, Z69, Z70, Z71: value 74LS74 -> 7474; footprint (none) -> Package_DIP:DIP-14_W7.62mm_Socket
- Z33: value 74LS10 -> 7410; footprint (none) -> Package_DIP:DIP-14_W7.62mm_Socket
- Z48: renamed from U48; value 74LS05 -> 7405; footprint (none) -> Package_DIP:DIP-14_W7.62mm_Socket; symbol 74xx:74LS05 -> Datapoint2200:74LS05
- Z48: value 74LS05 -> 7405; footprint (none) -> Package_DIP:DIP-14_W7.62mm_Socket; symbol 74xx:74LS05 -> Datapoint2200:74LS05
- Z50: value 74LS37 -> 7437; footprint (none) -> Package_DIP:DIP-14_W7.62mm_Socket
- Z51: value 74LS02 -> 7402; footprint (none) -> Package_DIP:DIP-14_W7.62mm_Socket
- Z59: value 74LS06 -> 7406; footprint (none) -> Package_DIP:DIP-14_W7.62mm_Socket; symbol 74xx:74LS06 -> Datapoint2200:74LS06
- Z59: renamed from U59; value 74LS06 -> 7406; footprint (none) -> Package_DIP:DIP-14_W7.62mm_Socket; symbol 74xx:74LS06 -> Datapoint2200:74LS06
- Z87: value 74LS73 -> 7473; footprint (none) -> Package_DIP:DIP-14_W7.62mm_Socket
Connections:
- net +5V: now also R53.2; no longer R53.1
- net DIV64_CLK: now also C54.1
- net GND: now also C54.2
- net ~WORD_SELECT: now also J901.1 (Pin_1)
- net ~EXECUTE: now reaches Z32.8 (~Q), Z50.10, Z50.12, Z51.11
- net at Z48.6, Z48.8, Z71.1 (~R)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: now also R53.1; no longer R53.2
- net ~KICK_START: now reaches Z71.4 (~S), Z71.8 (~Q)
- net ~NEXT_OPCODE: now reaches Z33.6, Z71.3 (C)
- net NEXT_IS_FETCH: now reaches Z70.12 (D), Z71.5 (Q)
- net ~RD_OPCODE: now reaches Z14.12, Z70.8 (~Q)
- net at Z87.10 (K), Z87.12 (Q), Z87.7 (J): now also Z115.10 (A0); no longer Z115.12 (A1)
- net at Z87.9 (Q): now also Z115.12 (A1); no longer Z115.10 (A0)
- net HALT renamed ~HALT
- net IR.CLK_EN renamed FETCH
- net JUMP_CALL_FLAG renamed JUMP_CALL_TAKE
- net MEM_OUTPUTS renamed ~DATA
- net OPCODE_ENABLE renamed DECODE_ENABLE
- net RUNNING renamed ~HALT_LIGHT
- net V renamed TEMP_ADDR.WR
- net ~IMM_RD renamed ~IND_RD
- net ~JUMP_CALL_FLAG renamed ~JUMP_CALL_TAKE
- net ~OPCODE_ENABLE renamed ~DECODE_ENABLE
- net ~RST_JUMP_CALL_FLAG renamed ~EXECUTE_DONE
- no-connect marks 7 -> 8
Other:
- note added: "!! The polarities of POR_IN and \nPOR_OUT can't *both* be inverted!"
- note added: "Clocks in A when\nduring fetch cycle\nReset when we start an \nexecute cycle whilst running"
- note added: "Clocks once\nper memory cycle"
- note added: "Data from tape\ndrives, sent whilst\nbooting."
- note added: "Data out from\nmemory cards."
- note added: "Data to memory\ncards"
- note added: "High whilst the second (high) byte\nof an inline address (for a jump or\ncall). (Into the temp addr reg)."
- note added: "If high the next WORD_SELECT\nwill initiaite a FETCH cycle.\n\n(High is only set at very end\nof execute cycle)"
- note added: "Internal data\nbus"
- note added: "Set during a fetch\ncycle. Clocking by\nWORD_SELECT\nensures memory is \nsync'ed"
- note added: "Set on booting, cleared \nshortly after. Forces a FETCH \ncycle into Z70B via Z70A"
- note added: "Starts execution of\nthe next opcode\n(if we're running)"
- note added: "To start the processor:\n* Cycle ~POR_IN\n* Hold RUN_SW high and EOR_REBOOT low\n* Cycle ~RESET_P low to clear address register\n* Wait for WORD_SELECT to go high\n* Send program data in via ~REBOOT_SERIAL_DATA\n(synced to PHI1_MEM and PHI2_MEM (not sure which))\n* Cycle EOR_REBOOT high.\nSystem should new be RUNNING and enter first FETCH cycle."
- note removed: "Cleared when booting \nor reading IR"
- note removed: "Cleared when booting \nor reading IR\nSet when finished reading IR\nClocks in running/halt state\nwhen we step a new instruction\n\nI.e. do we need a fetch or\nexecute cycle"
- note removed: "Clocks in A when\nwe start a fetch cycle\nReset when we start an \nexecute cycle whilst running"
- note removed: "Fetch (set)\nor execute (clear)"
- note removed: "High when /not/ reading into IR"
- note removed: "High when reading\ninto temp addr reg"
- note removed: "~Memory read/write required"
- note removed: "~Next instruction\n(step)??"
- moved on the sheet: C56, C57, R52, R53, R57, R58, R59, R60, R63, R64, R66, TP1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
